File: EAGLE/vr09-poc/vr09.sch (EAGLE design)
At the start: 18 parts

Commit message: wip
Parts:
- removed 0,0, 0,1, 0,2, 1,0, 1,1, 1,2, 2,0, 2,1, 2,2: KEYSWITCH-PLAIN-MX-1U, Keyboard:KEYSWITCH-PLAIN-MX-1U
- removed D0,0, D0,1, D0,2, D1,0, D1,1, D1,2, D2,0, D2,1, D2,2: (no value), Components:DIODE-SOD-123
- added D1, D2, D3, D4, D5, D6: (no value), diode:SCHOTTKY-DIODESMD
- added K00, K01, K02, K10, K11, K12: MX-5-PIN-HOTSWAP, ts_keyboards:MX-5-PIN-HOTSWAP
- added U$1, U$2, U$3, U$4, U$5, U$6: MX-FPRINT-1905-100U, ts_keyboards:MX-FPRINT-1905-100U
- added U$10, U$11, U$12, U$7, U$8, U$9: SK6812-E-REVERSE, ts_keyboards:SK6812-E-REVERSE
Connections:
- removed net ROW3: D0,2.C, D1,2.C, D2,2.C
- new net COL1: D1.C, D4.C
- new net COL2: D2.C, D5.C
- new net COL3: D3.C, D6.C
- new net GND: U$10.VSS_GND, U$11.VSS_GND, U$12.VSS_GND, U$7.VSS_GND, U$8.VSS_GND, U$9.VSS_GND
- new net N$1: U$7.DI
- new net N$10: U$10.DI, U$9.DO
- new net N$11: U$10.DO, U$11.DI
- new net N$12: U$11.DO, U$12.DI
- new net N$2: D4.A, K10.P
- new net N$3: D2.A, K01.P
- new net N$4: D1.A, K00.P
- new net N$5: D3.A, K02.P
- new net N$6: U$7.DO, U$8.DI
- new net N$7: D5.A, K11.P
- new net N$8: D6.A, K12.P
- new net N$9: U$8.DO, U$9.DI
- new net VCC: U$10.VDD, U$11.VDD, U$12.VDD, U$7.VDD, U$8.VDD, U$9.VDD
- net ROW1: now also K00.S, K01.S, K02.S; no longer D0,0.C, D1,0.C, D2,0.C
- net ROW2: now also K10.S, K11.S, K12.S; no longer D0,1.C, D1,1.C, D2,1.C

Commit message: wip
Parts:
- removed D1, D2, D3, D4, D5, D6: (no value), diode:SCHOTTKY-DIODESMD
- removed U$10, U$11, U$12, U$7, U$8, U$9: SK6812-E-REVERSE, ts_keyboards:SK6812-E-REVERSE
- added C00, C01, C02, C10, C11, C12: 100nF, rcl:C-EUC0603
- added D00, D01, D02, D10, D11, D12: (no value), jlcpcb_basic_parts:1N5819WS
- added L00, L01, L02, L10, L11, L12: SK6812-E-REVERSEDRILL, ts_keyboards:SK6812-E-REVERSEDRILL
- added R1: 500ohm, rcl:R-EU_R0603
Connections:
- removed net N$10: U$10.DI, U$9.DO
- removed net N$8: D6.A, K12.P
- removed net N$9: U$8.DO, U$9.DI
- new net DIN: R1.1
- new net N$13: L11.2_DOUT, L12.4_DIN
- new net N$14: L10.2_DOUT, L11.4_DIN
- new net N$19: L02.2_DOUT, L10.4_DIN
- net COL1: now also K00.P, K10.P; no longer D1.C, D4.C
- net COL2: now also K01.P, K11.P; no longer D2.C, D5.C
- net COL3: now also K02.P, K12.P; no longer D3.C, D6.C
- net GND: now also C00.2, C01.2, C02.2, C10.2, C11.2, C12.2, L00.3_GND, L01.3_GND, L02.3_GND, L10.3_GND, L11.3_GND, L12.3_GND; no longer U$10.VSS_GND, U$11.VSS_GND, U$12.VSS_GND, U$7.VSS_GND, U$8.VSS_GND, U$9.VSS_GND
- net N$1: now also D10.A, K10.S; no longer U$7.DI
- net N$11: now also L00.2_DOUT, L01.4_DIN; no longer U$10.DO, U$11.DI
- net N$12: now also L01.2_DOUT, L02.4_DIN; no longer U$11.DO, U$12.DI
- net N$2: now also D11.A, K11.S; no longer D4.A, K10.P
- net N$3: now also D12.A, K12.S; no longer D2.A, K01.P
- net N$4: now also D02.A, K02.S; no longer D1.A, K00.P
- net N$5: now also D01.A, K01.S; no longer D3.A, K02.P
- net N$6: now also L00.4_DIN, R1.2; no longer U$7.DO, U$8.DI
- net N$7: now also D00.A, K00.S; no longer D5.A, K11.P
- net ROW1: now also D00.C, D01.C, D02.C; no longer K00.S, K01.S, K02.S
- net ROW2: now also D10.C, D11.C, D12.C; no longer K10.S, K11.S, K12.S
- net VCC: now also C00.1, C01.1, C02.1, C10.1, C11.1, C12.1, L00.1_VDD, L01.1_VDD, L02.1_VDD, L10.1_VDD, L11.1_VDD, L12.1_VDD; no longer U$10.VDD, U$11.VDD, U$12.VDD, U$7.VDD, U$8.VDD, U$9.VDD

Commit message: wip
Parts:
- added J1: MICROMOD-2222-C, SparkFun-MicroMod:MICROMOD-2222-C
- U$3: value MX-FPRINT-1905-100U -> MX-FPRINT-1905-200U; device ts_keyboards:MX-FPRINT-1905-100U -> ts_keyboards:MX-FPRINT-1905-200U
- U$4, U$6: value MX-FPRINT-1905-100U -> MX-FPRINT-1905-150U; device ts_keyboards:MX-FPRINT-1905-100U -> ts_keyboards:MX-FPRINT-1905-150U
Changed lines of the file:
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@@
 <part name="U$1" library="ts_keyboards" deviceset="MX-FPRINT-1905-100U" device=""/>
 <part name="U$2" library="ts_keyboards" deviceset="MX-FPRINT-1905-100U" device=""/>
-<part name="U$3" library="ts_keyboards" deviceset="MX-FPRINT-1905-100U" device=""/>
-<part name="U$4" library="ts_keyboards" deviceset="MX-FPRINT-1905-100U" device=""/>
 <part name="U$5" library="ts_keyboards" deviceset="MX-FPRINT-1905-100U" device=""/>
-<part name="U$6" library="ts_keyboards" deviceset="MX-FPRINT-1905-100U" device=""/>
 <part name="D00" library="jlcpcb_basic_parts" deviceset="1N5819WS" device=""/>
 <part name="D01" library="jlcpcb_basic_parts" deviceset="1N5819WS" device=""/>
@@
 <part name="GND2" library="ts_custom_nick_nacks" deviceset="GND" device=""/>
 <part name="R1" library="rcl" library_urn="urn:adsk.eagle:library:334" deviceset="R-EU_" device="R0603" package3d_urn="urn:adsk.eagle:package:23555/3" value="500ohm"/>
+<part name="J1" library="SparkFun-MicroMod" deviceset="MICROMOD" device="-2222-C"/>
+<part name="U$3" library="ts_keyboards" deviceset="MX-FPRINT-1905-200U" device=""/>
+<part name="U$4" library="ts_keyboards" deviceset="MX-FPRINT-1905-150U" device=""/>
+<part name="U$6" library="ts_keyboards" deviceset="MX-FPRINT-1905-150U" device=""/>
 </parts>
 <sheets>
@@
 <instance part="U$1" gate="G$1" x="35.56" y="139.7" smashed="yes"/>
 <instance part="U$2" gate="G$1" x="60.96" y="139.7" smashed="yes"/>
-<instance part="U$3" gate="G$1" x="86.36" y="139.7" smashed="yes"/>
-<instance part="U$4" gate="G$1" x="35.56" y="106.68" smashed="yes"/>
 <instance part="U$5" gate="G$1" x="60.96" y="106.68" smashed="yes"/>
-<instance part="U$6" gate="G$1" x="86.36" y="106.68" smashed="yes"/>
 <instance part="D00" gate="G$1" x="48.26" y="144.78" smashed="yes" rot="R270">
 <attribute name="NAME" x="50.165" y="147.066" size="1.778" layer="95" rot="R270"/>
@@
 <attribute name="VALUE" x="26.67" y="67.818" size="1.778" layer="96"/>
 </instance>
+<instance part="J1" gate="J1" x="223.52" y="104.14" smashed="yes">
+<attribute name="NAME" x="203.2" y="157.988" size="1.778" layer="95"/>
+<attribute name="VALUE" x="203.2" y="55.88" size="1.778" layer="96"/>
+</instance>
+<instance part="U$3" gate="G$1" x="86.36" y="139.7" smashed="yes"/>
+<instance part="U$4" gate="G$1" x="35.56" y="106.68" smashed="yes"/>
+<instance part="U$6" gate="G$1" x="86.36" y="106.68" smashed="yes"/>
 </instances>
 <busses>
@@
 </drawing>
 <compatibility>
+<note version="6.3" minversion="6.2.2" severity="warning">
+Since Version 6.2.2 text objects can contain more than one line,
+which will not be processed correctly with this version.
+</note>
 <note version="8.2" severity="warning">
 Since Version 8.2, EAGLE supports online libraries. The ids
