File: EAGLE/vr60-keyboard/vr60.sch (EAGLE design)
At the start: 0 parts

Commit message: wip
Parts:
- added D1, D10, D11, D12, D13, D14, D15, D16, D17, D18, D19, D2, D20, D21, D22, D23, D24, D25, D26, D27, D28, D29, D3, D30, D31, D32, D33, D34, D35, D36, D37, D38, D39, D4, D40, D41, D42, D43, D44, D45, D46, D47, D48, D49, D5, D50, D51, D52, D53, D54, D55, D56, D57, D58, D59, D6, D60, D61, D7, D8, D9: (no value), jlcpcb_basic_parts:1N5819WS
- added U$1, U$10, U$11, U$12, U$13, U$14, U$15, U$16, U$17, U$18, U$19, U$2, U$20, U$21, U$22, U$23, U$24, U$25, U$26, U$27, U$28, U$29, U$3, U$30, U$31, U$32, U$33, U$34, U$35, U$36, U$37, U$38, U$39, U$4, U$40, U$41, U$42, U$43, U$44, U$45, U$46, U$47, U$48, U$49, U$5, U$50, U$51, U$52, U$53, U$54, U$55, U$56, U$57, U$58, U$59, U$6, U$60, U$61, U$7, U$8, U$9: MX-5-PIN-HOTSWAP, ts_keyboards:MX-5-PIN-HOTSWAP
Connections:
- new net COL00: D1.C, D15.C, D29.C, D42.C, D54.C
- new net COL01: D16.C, D2.C, D30.C, D55.C
- new net COL02: D17.C, D3.C, D31.C, D43.C, D56.C
- new net COL03: D18.C, D32.C, D4.C, D44.C
- new net COL04: D19.C, D33.C, D45.C, D5.C
- new net COL05: D20.C, D34.C, D46.C, D6.C
- new net COL06: D21.C, D35.C, D47.C, D57.C, D7.C
- new net COL07: D22.C, D36.C, D48.C, D8.C
- new net COL08: D23.C, D37.C, D49.C, D9.C
- new net COL09: D10.C, D24.C, D38.C, D50.C
- new net COL10: D11.C, D25.C, D39.C, D51.C, D58.C
- new net COL11: D12.C, D26.C, D40.C, D52.C, D59.C
- new net COL12: D13.C, D27.C, D60.C
- new net COL13: D14.C, D28.C, D41.C, D53.C, D61.C
- new net N$1: D1.A, U$1.P
- new net N$10: D10.A, U$10.P
- new net N$11: D11.A, U$11.P
- new net N$12: D12.A, U$12.P
- new net N$13: D13.A, U$13.P
- new net N$14: D14.A, U$14.P
- new net N$15: D15.A, U$15.P
- new net N$16: D16.A, U$16.P
- new net N$17: D17.A, U$17.P
- new net N$18: D18.A, U$18.P
- new net N$19: D19.A, U$19.P
- new net N$2: D2.A, U$2.P
- new net N$20: D20.A, U$20.P
- new net N$21: D21.A, U$21.P
- new net N$22: D22.A, U$22.P
- new net N$23: D23.A, U$23.P
- new net N$24: D24.A, U$24.P
- new net N$25: D25.A, U$25.P
- new net N$26: D26.A, U$26.P
- new net N$27: D27.A, U$27.P
- new net N$28: D28.A, U$28.P
- new net N$29: D29.A, U$29.P
- new net N$3: D3.A, U$3.P
- new net N$30: D30.A, U$30.P
- new net N$31: D31.A, U$31.P
- new net N$32: D32.A, U$32.P
- new net N$33: D33.A, U$33.P
- new net N$34: D34.A, U$34.P
- new net N$35: D35.A, U$35.P
- new net N$36: D36.A, U$36.P
- new net N$37: D37.A, U$37.P
- new net N$38: D38.A, U$38.P
- new net N$39: D39.A, U$39.P
- new net N$4: D4.A, U$4.P
- new net N$40: D40.A, U$40.P
- new net N$41: D41.A, U$41.P
- new net N$42: D42.A, U$42.P
- new net N$43: D43.A, U$43.P
- new net N$44: D44.A, U$44.P
- new net N$45: D45.A, U$45.P
- new net N$46: D46.A, U$46.P
- new net N$47: D47.A, U$47.P
- new net N$48: D48.A, U$48.P
- new net N$49: D49.A, U$49.P
- new net N$5: D5.A, U$5.P
- new net N$50: D50.A, U$50.P
- new net N$51: D51.A, U$51.P
- new net N$52: D52.A, U$52.P
- new net N$53: D53.A, U$53.P
- new net N$54: D54.A, U$54.P
- new net N$55: D55.A, U$55.P
- new net N$56: D56.A, U$56.P
- new net N$57: D57.A, U$57.P
- new net N$58: D58.A, U$58.P
- new net N$59: D59.A, U$59.P
- new net N$6: D6.A, U$6.P
- new net N$60: D60.A, U$60.P
- new net N$61: D61.A, U$61.P
- new net N$7: D7.A, U$7.P
- new net N$8: D8.A, U$8.P
- new net N$9: D9.A, U$9.P
- new net ROW0: U$1.S, U$10.S, U$11.S, U$12.S, U$13.S, U$14.S, U$2.S, U$3.S, U$4.S, U$5.S, U$6.S, U$7.S, U$8.S, U$9.S
- new net ROW1: U$15.S, U$16.S, U$17.S, U$18.S, U$19.S, U$20.S, U$21.S, U$22.S, U$23.S, U$24.S, U$25.S, U$26.S, U$27.S, U$28.S
- new net ROW2: U$29.S, U$30.S, U$31.S, U$32.S, U$33.S, U$34.S, U$35.S, U$36.S, U$37.S, U$38.S, U$39.S, U$40.S, U$41.S
- new net ROW3: U$42.S, U$43.S, U$44.S, U$45.S, U$46.S, U$47.S, U$48.S, U$49.S, U$50.S, U$51.S, U$52.S, U$53.S
- new net ROW4: U$54.S, U$55.S, U$56.S, U$57.S, U$58.S, U$59.S, U$60.S, U$61.S
