File: EAGLE/vr60-micromod/vr60.sch (EAGLE design)
At the start: 122 parts

Commit message: wip
Parts:
- added B14, B41, B42, B53: MX-STABS-200U, ts_keyboards:MX-STABS-200U
- added B57: MX-STABS-625U, ts_keyboards:MX-STABS-625U
- added Z1, Z10, Z11, Z12, Z13, Z16, Z17, Z18, Z19, Z2, Z20, Z21, Z22, Z23, Z24, Z25, Z26, Z27, Z3, Z30, Z31, Z32, Z33, Z34, Z35, Z36, Z37, Z38, Z39, Z4, Z40, Z43, Z44, Z45, Z46, Z47, Z48, Z49, Z5, Z50, Z51, Z52, Z6, Z7, Z8, Z9: MX-FPRINT-100U19, ts_keyboards:MX-FPRINT-100U19
- added Z14: MX-FPRINT-200U19, ts_keyboards:MX-FPRINT-200U19
- added Z15, Z28: MX-FPRINT-150U19, ts_keyboards:MX-FPRINT-150U19
- added Z29: MX-FPRINT-175U19, ts_keyboards:MX-FPRINT-175U19
- added Z41, Z42: MX-FPRINT-225U19, ts_keyboards:MX-FPRINT-225U19
- added Z53: MX-FPRINT-275U19, ts_keyboards:MX-FPRINT-275U19
- added Z54, Z55, Z56, Z58, Z59, Z60, Z61: MX-FPRINT-125U19, ts_keyboards:MX-FPRINT-125U19
- added Z57: MX-FPRINT-625U19, ts_keyboards:MX-FPRINT-625U19
- renumbered U$1 to S1, U$10 to S10, U$11 to S11, U$12 to S12, U$13 to S13, U$14 to S14, U$15 to S15, U$16 to S16, U$17 to S17, U$18 to S18, U$19 to S19, U$2 to S2, U$20 to S20, U$21 to S21, U$22 to S22, U$23 to S23, U$24 to S24, U$25 to S25, U$26 to S26, U$27 to S27, U$28 to S28, U$29 to S29, U$3 to S3, U$30 to S30, U$31 to S31, U$32 to S32, U$33 to S33, U$34 to S34, U$35 to S35, U$36 to S36, U$37 to S37, U$38 to S38, U$39 to S39, U$4 to S4, U$40 to S40, U$41 to S41, U$42 to S42, U$43 to S43, U$44 to S44, U$45 to S45, U$46 to S46, U$47 to S47, U$48 to S48, U$49 to S49, U$5 to S5, U$50 to S50, U$51 to S51, U$52 to S52, U$53 to S53, U$54 to S54, U$55 to S55, U$56 to S56, U$57 to S57, U$58 to S58, U$59 to S59, U$6 to S6, U$60 to S60, U$61 to S61, U$7 to S7, U$8 to S8, U$9 to S9
Connections:
- net COL00 renamed COL0
- net COL01 renamed COL1
- net COL02 renamed COL2
- net COL03 renamed COL3
- net COL04 renamed COL4
- net COL05 renamed COL5
- net COL06 renamed COL6
- net COL07 renamed COL7
- net COL08 renamed COL8
- net COL09 renamed COL9
