File: EAGLE/vr60-micromod/vr60.brd (EAGLE design)
At the start: 285 x 94.6 mm, 122 parts

Commit message: wip
Parts:
- added B14, B41, B42, B53: MX-STABS-200U, ts_keyboards:MX-STABS-200U
- added B57: MX-STABS-625U, ts_keyboards:MX-STABS-625U
- added Z1, Z10, Z11, Z12, Z13, Z16, Z17, Z18, Z19, Z2, Z20, Z21, Z22, Z23, Z24, Z25, Z26, Z27, Z3, Z30, Z31, Z32, Z33, Z34, Z35, Z36, Z37, Z38, Z39, Z4, Z40, Z43, Z44, Z45, Z46, Z47, Z48, Z49, Z5, Z50, Z51, Z52, Z6, Z7, Z8, Z9: MX-FPRINT-100U19, ts_keyboards:MX-FPRINT-1900-100U
- added Z14: MX-FPRINT-200U19, ts_keyboards:MX-FPRINT-1900-200U
- added Z15, Z28: MX-FPRINT-150U19, ts_keyboards:MX-FPRINT-1900-150U
- added Z29: MX-FPRINT-175U19, ts_keyboards:MX-FPRINT-1900-175U
- added Z41, Z42: MX-FPRINT-225U19, ts_keyboards:MX-FPRINT-1900-225U
- added Z53: MX-FPRINT-275U19, ts_keyboards:MX-FPRINT-1900-275U
- added Z54, Z55, Z56, Z58, Z59, Z60, Z61: MX-FPRINT-125U19, ts_keyboards:MX-FPRINT-1900-125U
- added Z57: MX-FPRINT-625U19, ts_keyboards:MX-FPRINT-1900-625U
- renumbered U$1 to S1, U$10 to S10, U$11 to S11, U$12 to S12, U$13 to S13, U$14 to S14, U$15 to S15, U$16 to S16, U$17 to S17, U$18 to S18, U$19 to S19, U$2 to S2, U$20 to S20, U$21 to S21, U$22 to S22, U$23 to S23, U$24 to S24, U$25 to S25, U$26 to S26, U$27 to S27, U$28 to S28, U$29 to S29, U$3 to S3, U$30 to S30, U$31 to S31, U$32 to S32, U$33 to S33, U$34 to S34, U$35 to S35, U$36 to S36, U$37 to S37, U$38 to S38, U$39 to S39, U$4 to S4, U$40 to S40, U$41 to S41, U$42 to S42, U$43 to S43, U$44 to S44, U$45 to S45, U$46 to S46, U$47 to S47, U$48 to S48, U$49 to S49, U$5 to S5, U$50 to S50, U$51 to S51, U$52 to S52, U$53 to S53, U$54 to S54, U$55 to S55, U$56 to S56, U$57 to S57, U$58 to S58, U$59 to S59, U$6 to S6, U$60 to S60, U$61 to S61, U$7 to S7, U$8 to S8, U$9 to S9
Connections:
- net COL00 renamed COL0
- net COL01 renamed COL1
- net COL02 renamed COL2
- net COL03 renamed COL3
- net COL04 renamed COL4
- net COL05 renamed COL5
- net COL06 renamed COL6
- net COL07 renamed COL7
- net COL08 renamed COL8
- net COL09 renamed COL9

Commit message: wip
Parts:
- moved B53 1731.2 mm to (258.9, 28.5), turned to 180 degrees
- moved B14 1730.3 mm to (266.0, 85.5), turned to 180 degrees
- moved B41 1712.3 mm to (263.6, 47.5), turned to 180 degrees
- moved B57 1694.7 mm to (130.6, 9.50)
- moved B42 1662.7 mm to (21.4, 28.5), turned to 180 degrees
- moved Z61 1640.9 mm to (273.1, 9.50)
- moved Z60 1614.8 mm to (249.4, 9.50)
- moved Z59 1589.0 mm to (225.6, 9.50)
- moved Z58 1563.3 mm to (201.9, 9.50)
- moved Z57 1516.6 mm to (130.6, 9.50)
- moved Z53 1497.9 mm to (258.9, 28.5)
- moved Z56 1492.4 mm to (59.4, 9.50)
- moved Z52 1472.9 mm to (223.2, 28.5)
- moved Z55 1468.5 mm to (35.6, 9.50)
- moved Z51 1448.2 mm to (204.2, 28.5)
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
Commit message: wip
Other:
- board size 285 x 94.6 mm -> 283 x 93 mm
- board text added: "AP-3 x136.2 y57.9 d2.5"
Changed lines of the file:
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@@
 <?xml version="1.0" encoding="utf-8"?>
 <!DOCTYPE eagle SYSTEM "eagle.dtd">
-<eagle version="9.5.1">
+<eagle version="9.6.2">
 <drawing>
 <settings>
-<setting alwaysvectorfont="no"/>
+<setting alwaysvectorfont="yes"/>
 <setting verticaltext="up"/>
 </settings>
@@
 <board>
 <plain>
-<wire x1="1" y1="0" x2="284" y2="0" width="0" layer="20"/>
-<hole x="260.05" y="66.7" drill="3" locked="yes"/>
-<hole x="25.2" y="66.7" drill="3" locked="yes"/>
-<hole x="128.2" y="47.6" drill="3" locked="yes"/>
-<hole x="190.5" y="9.3" drill="3" locked="yes"/>
-<hole x="3" y="38.1" drill="3" locked="yes"/>
-<hole x="282" y="38.1" drill="3"/>
-<hole x="25" y="65.8" drill="3" locked="yes"/>
-<hole x="260" y="65.8" drill="3"/>
-<hole x="136" y="56.8" drill="3" locked="yes"/>
-<hole x="237" y="20.8" drill="3" locked="yes"/>
-<hole x="74" y="15.8" drill="3" locked="yes"/>
-<wire x1="285" y1="1" x2="285" y2="36.6" width="0" layer="20"/>
-<wire x1="285" y1="39.6" x2="285" y2="93.6" width="0" layer="20"/>
-<wire x1="284" y1="94.6" x2="1" y2="94.6" width="0" layer="20"/>
-<wire x1="0" y1="93.6" x2="0" y2="39.6" width="0" layer="20"/>
-<wire x1="0" y1="36.6" x2="0" y2="1" width="0" layer="20"/>
-<wire x1="0" y1="93.6" x2="1" y2="94.6" width="0" layer="20" curve="-90"/>
-<wire x1="1" y1="0" x2="0" y2="1" width="0" layer="20" curve="-90"/>
-<wire x1="284" y1="94.6" x2="285" y2="93.6" width="0" layer="20" curve="-90"/>
-<wire x1="285" y1="1" x2="284" y2="0" width="0" layer="20" curve="-90"/>
-<wire x1="3" y1="39.6" x2="3" y2="36.6" width="0" layer="20" curve="-180"/>
-<wire x1="3" y1="39.6" x2="0" y2="39.6" width="0" layer="20"/>
-<wire x1="3" y1="36.6" x2="0" y2="36.6" width="0" layer="20"/>
-<wire x1="282" y1="36.6" x2="282" y2="39.6" width="0" layer="20" curve="-180"/>
-<wire x1="282" y1="39.6" x2="285" y2="39.6" width="0" layer="20"/>
-<wire x1="282" y1="36.6" x2="285" y2="36.6" width="0" layer="20"/>
-<circle x="29.15" y="46.4" radius="3.5" width="0.5" layer="22"/>
+<hole x="128.2" y="47.6" drill="3"/>
+<wire x1="0" y1="0" x2="0" y2="95" width="0.1524" layer="48"/>
+<wire x1="0" y1="95" x2="285" y2="95" width="0.1524" layer="48"/>
+<wire x1="285" y1="95" x2="285" y2="0" width="0.1524" layer="48"/>
+<wire x1="285" y1="0" x2="0" y2="0" width="0.1524" layer="48"/>
+<hole x="25.2" y="66.9" drill="2.5" locked="yes"/>
+<hole x="260.05" y="66.9" drill="2.5" locked="yes"/>
+<hole x="128.2" y="47.8" drill="2.5" locked="yes"/>
+<hole x="2.5" y="38.3" drill="2.5" locked="yes"/>
+<hole x="282.5" y="38.3" drill="2.5" locked="yes"/>
+<hole x="190.5" y="9.6" drill="2.5" locked="yes"/>
+<wire x1="284" y1="92" x2="284" y2="3" width="0.1524" layer="20"/>
+<wire x1="284" y1="3" x2="282" y2="1" width="0.1524" layer="20" curve="-90"/>
+<wire x1="282" y1="1" x2="3" y2="1" width="0.1524" layer="20"/>
+<wire x1="3" y1="1" x2="1" y2="3" width="0.1524" layer="20" curve="-90"/>
+<wire x1="1" y1="3" x2="1" y2="92" width="0.1524" layer="20"/>
+<wire x1="1" y1="92" x2="3" y2="94" width="0.1524" layer="20" curve="-90"/>
+<wire x1="3" y1="94" x2="282" y2="94" width="0.1524" layer="20"/>
+<wire x1="282" y1="94" x2="284" y2="92" width="0.1524" layer="20" curve="-90"/>
+<hole x="136.2" y="57.9" drill="2.5" locked="yes"/>
+<hole x="74.2" y="16.9" drill="2.5" locked="yes"/>
+<hole x="237.2" y="21.9" drill="2.5" locked="yes"/>
+<text x="135" y="60" size="1.778" layer="48">AP-3
+x136.2 y57.9 d2.5</text>
+<wire x1="28.7" y1="48.9" x2="32.7" y2="48.9" width="0.01" layer="49"/>
+<wire x1="32.7" y1="48.9" x2="32.7" y2="46.9" width="0.01" layer="49"/>
+<wire x1="32.7" y1="46.9" x2="28.7" y2="46.9" width="0.01" layer="49"/>
+<wire x1="28.7" y1="46.9" x2="28.7" y2="48.9" width="0.01" layer="49"/>
+<wire x1="34.2" y1="57.9" x2="34.2" y2="87.9" width="0.01" layer="49" style="shortdash"/>
+<wire x1="34.2" y1="87.9" x2="119.2" y2="87.9" width="0.01" layer="49" style="shortdash"/>
+<wire x1="119.2" y1="87.9" x2="119.2" y2="57.9" width="0.01" layer="49" style="shortdash"/>
+<wire x1="119.2" y1="57.9" x2="34.2" y2="57.9" width="0.01" layer="49" style="shortdash"/>
+<wire x1="18.2" y1="96" x2="18.2" y2="85" width="0.01" layer="49" style="dashdot"/>
+<wire x1="13.7" y1="94" x2="13.7" y2="87" width="0.01" layer="49" style="shortdash"/>
+<wire x1="13.7" y1="87" x2="22.7" y2="87" width="0.01" layer="49" style="shortdash"/>
+<wire x1="22.7" y1="87" x2="22.7" y2="94" width="0.01" layer="49" style="shortdash"/>
+<circle x="29.15" y="46.6" radius="2.5" width="0.01" layer="49"/>
 </plain>
 <attributes>
@@
 </drawing>
 <compatibility>
+<note version="6.3" minversion="6.2.2" severity="warning">
+Since Version 6.2.2 text objects can contain more than one line,
+which will not be processed correctly with this version.
+</note>
 <note version="8.5" severity="warning">
 Since Version 8.5, EAGLE supports locking for holes, vias, wires and polygons.
