File: EAGLE/vr61/vr60.brd (EAGLE design)
At the start: 283 x 93 mm, 188 parts

Commit message: .
Parts:
- added H5: STAND-OFF-REFLOW2.5MM_TALL, SparkFun-Hardware:STAND-OFF-REFLOW-M2.5
- added J6: MICROMOD-2222-C, SparkFun-MicroMod:M.2-CONNECTOR-E
- moved D29 19.0 mm to (4.75, 51.0)
- moved D15 17.0 mm to (4.38, 70.0)
- turned S-EQL to 0 degrees
- turned S_0 to 0 degrees
- turned S_2 to 0 degrees
- turned S_3 to 0 degrees
- turned S_4 to 0 degrees
- turned S_5 to 0 degrees
- turned S_6 to 0 degrees
- turned S_7 to 0 degrees
- turned S_8 to 0 degrees
- turned S_9 to 0 degrees
- turned S_A to 0 degrees
- turned S_B to 0 degrees
- turned S_BSL to 0 degrees
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- renumbered S1 to S_ESC, S10 to S_9, S11 to S_0, S12 to S_MIN, S13 to S-EQL, S14 to S_BSP, S15 to S_TAB, S16 to S_Q, S17 to S_W, S18 to S_E, S19 to S_R, S2 to S_1, S20 to S_T, S21 to S_Y, S22 to S_U, S23 to S_I, S24 to S_O, S25 to S_P, S26 to S_OB, S27 to S_CB, S28 to S_BSL, S29 to S_CPS, S3 to S_2, S30 to S_A, S31 to S_S, S32 to S_D, S33 to S_F, S34 to S_G, S35 to S_H, S36 to S_J, S37 to S_K, S38 to S_L, S39 to S_SCL, S4 to S_3, S40 to S_QUO, S41 to S_ENT, S42 to S_LSH, S43 to S_Z, S44 to S_X, S45 to S_C, S46 to S_V, S47 to S_B, S48 to S_N, S49 to S_M, S5 to S_4, S50 to S_COM, S51 to S_DOT, S52 to S_FSL, S53 to S_RSH, S54 to S_LCT, S55 to S_LGU, S56 to S_LAL, S57 to S_SPC, S58 to S_FN1, S59 to S_RAL, S6 to S_5, S60 to S_RGU, S61 to S_RCT, S7 to S_6, S8 to S_7, S9 to S_8
Connections:
- removed net COL10: D11.C, D25.C, D39.C, D51.C, D58.C
- removed net COL11: D12.C, D26.C, D40.C, D52.C, D59.C
- removed net COL12: D13.C, D27.C, D60.C
- removed net COL13: D14.C, D28.C, D41.C, D53.C, D61.C
- removed net COL8: D23.C, D37.C, D49.C, D9.C
- removed net COL9: D10.C, D24.C, D38.C, D50.C
- new net GND: H5.1
- new net ROW5: S-EQL.P$2, S_0.P$2, S_8.P$2, S_9.P$2, S_BSP.P$2, S_MIN.P$2
- new net ROW6: S_BSL.P$2, S_CB.P$2, S_I.P$2, S_O.P$2, S_OB.P$2, S_P.P$2
- new net ROW7: S_ENT.P$2, S_K.P$2, S_L.P$2, S_QUO.P$2, S_SCL.P$2
- new net ROW8: S_COM.P$2, S_DOT.P$2, S_FSL.P$2, S_M.P$2, S_RSH.P$2
- net COL0: now also D23.C, D37.C, D49.C, D9.C
- net COL1: now also D10.C, D24.C, D38.C, D50.C
- net COL2: now also D11.C, D25.C, D39.C, D51.C
- net COL3: now also D12.C, D26.C, D40.C, D52.C, D57.C
- net COL4: now also D13.C, D27.C, D58.C
- net COL5: now also D53.C, D59.C
- net COL6: now also D14.C, D28.C, D41.C, D60.C; no longer D57.C
- net COL7: now also D61.C
- net ROW0: no longer S-EQL.P$2, S_0.P$2, S_8.P$2, S_9.P$2, S_BSP.P$2, S_MIN.P$2
- net ROW1: no longer S_BSL.P$2, S_CB.P$2, S_I.P$2, S_O.P$2, S_OB.P$2, S_P.P$2
- net ROW2: no longer S_ENT.P$2, S_K.P$2, S_L.P$2, S_QUO.P$2, S_SCL.P$2
- net ROW3: no longer S_COM.P$2, S_DOT.P$2, S_FSL.P$2, S_M.P$2, S_RSH.P$2

Commit message: .
Parts:
- moved D4 19.7 mm to (58.0, 78.0), turned to 90 degrees
- moved D28 18.4 mm to (263.1, 60.0), turned to 90 degrees
- moved D41 18.2 mm to (253.2, 47.0), turned to 90 degrees
- moved D3 12.0 mm to (55.0, 78.0), turned to 90 degrees
- moved D5 9.10 mm to (94.0, 81.0), turned to 90 degrees
- moved D14 4.93 mm to (276.0, 86.0), turned to 0 degrees
- moved D1 4.65 mm to (19.0, 86.0), turned to 0 degrees
- moved D10 4.65 mm to (190.0, 86.0), turned to 0 degrees
- moved D11 4.65 mm to (209.0, 86.0), turned to 0 degrees
- moved D12 4.65 mm to (228.0, 86.0), turned to 0 degrees
- moved D13 4.65 mm to (247.0, 86.0), turned to 0 degrees
- moved D2 4.65 mm to (38.0, 86.0), turned to 0 degrees
- moved D6 4.65 mm to (114.0, 86.0), turned to 0 degrees
- moved D7 4.65 mm to (133.0, 86.0), turned to 0 degrees
- moved D8 4.65 mm to (152.0, 86.0), turned to 0 degrees
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Connections:
- removed net COL0: D1.C, D15.C, D23.C, D29.C, D37.C, D42.C, D49.C, D54.C, D9.C
- removed net COL1: D10.C, D16.C, D2.C, D24.C, D30.C, D38.C, D50.C, D55.C
- removed net COL2: D11.C, D17.C, D25.C, D3.C, D31.C, D39.C, D43.C, D51.C, D56.C
- removed net COL3: D12.C, D18.C, D26.C, D32.C, D4.C, D40.C, D44.C, D52.C, D57.C
- removed net COL4: D13.C, D19.C, D27.C, D33.C, D45.C, D5.C, D58.C
- removed net COL5: D20.C, D34.C, D46.C, D53.C, D59.C, D6.C
- removed net COL6: D14.C, D21.C, D28.C, D35.C, D41.C, D47.C, D60.C, D7.C
- removed net COL7: D22.C, D36.C, D48.C, D61.C, D8.C
- removed net ROW0: S_1.P$2, S_2.P$2, S_3.P$2, S_4.P$2, S_5.P$2, S_6.P$2, S_7.P$2, S_ESC.P$2
- removed net ROW1: S_E.P$2, S_Q.P$2, S_R.P$2, S_T.P$2, S_TAB.P$2, S_U.P$2, S_W.P$2, S_Y.P$2
- removed net ROW2: S_A.P$2, S_CPS.P$2, S_D.P$2, S_F.P$2, S_G.P$2, S_H.P$2, S_J.P$2, S_S.P$2
- removed net ROW3: S_B.P$2, S_C.P$2, S_LSH.P$2, S_N.P$2, S_V.P$2, S_X.P$2, S_Z.P$2
- removed net ROW4: S_FN1.P$2, S_LAL.P$2, S_LCT.P$2, S_LGU.P$2, S_RAL.P$2, S_RCT.P$2, S_RGU.P$2, S_SPC.P$2
- removed net ROW5: S-EQL.P$2, S_0.P$2, S_8.P$2, S_9.P$2, S_BSP.P$2, S_MIN.P$2
- removed net ROW6: S_BSL.P$2, S_CB.P$2, S_I.P$2, S_O.P$2, S_OB.P$2, S_P.P$2
- removed net ROW7: S_ENT.P$2, S_K.P$2, S_L.P$2, S_QUO.P$2, S_SCL.P$2
- removed net ROW8: S_COM.P$2, S_DOT.P$2, S_FSL.P$2, S_M.P$2, S_RSH.P$2
- new net MX0: D1.C, D15.C, D23.C, D29.C, D37.C, D42.C, D49.C, D54.C, D9.C, J6.18
- new net MX1: D10.C, D16.C, D2.C, D24.C, D30.C, D38.C, D50.C, D55.C, J6.16
- new net MX2: D11.C, D17.C, D25.C, D3.C, D31.C, D39.C, D43.C, D51.C, D56.C, J6.14
- new net MX3: D12.C, D18.C, D26.C, D32.C, D4.C, D40.C, D44.C, D52.C, D57.C, J6.38
- new net MX4: D13.C, D19.C, D27.C, D33.C, D45.C, D5.C, D58.C, J6.12
- new net MX5: D20.C, D34.C, D46.C, D53.C, D59.C, D6.C, J6.10
- new net MX6: D14.C, D21.C, D28.C, D35.C, D41.C, D47.C, D60.C, D7.C, J6.17
- new net MX7: D22.C, D36.C, D48.C, D61.C, D8.C, J6.19
- new net MY0: J6.56, S_1.P$2, S_2.P$2, S_3.P$2, S_4.P$2, S_5.P$2, S_6.P$2, S_7.P$2, S_ESC.P$2
- new net MY1: J6.54, S_E.P$2, S_Q.P$2, S_R.P$2, S_T.P$2, S_TAB.P$2, S_U.P$2, S_W.P$2, S_Y.P$2
- new net MY2: J6.52, S_A.P$2, S_CPS.P$2, S_D.P$2, S_F.P$2, S_G.P$2, S_H.P$2, S_J.P$2, S_S.P$2
- new net MY3: J6.50, S_B.P$2, S_C.P$2, S_LSH.P$2, S_N.P$2, S_V.P$2, S_X.P$2, S_Z.P$2
- new net MY4: J6.48, S_FN1.P$2, S_LAL.P$2, S_LCT.P$2, S_LGU.P$2, S_RAL.P$2, S_RCT.P$2, S_RGU.P$2, S_SPC.P$2
- new net MY5: J6.46, S-EQL.P$2, S_0.P$2, S_8.P$2, S_9.P$2, S_BSP.P$2, S_MIN.P$2
- new net MY6: J6.44, S_BSL.P$2, S_CB.P$2, S_I.P$2, S_O.P$2, S_OB.P$2, S_P.P$2
- new net MY7: J6.42, S_ENT.P$2, S_K.P$2, S_L.P$2, S_QUO.P$2, S_SCL.P$2
- new net MY8: J6.40, S_COM.P$2, S_DOT.P$2, S_FSL.P$2, S_M.P$2, S_RSH.P$2
- new net VCC: J6.2, J6.74
- net GND: now also J6.1, J6.33, J6.36, J6.39, J6.45, J6.7, J6.75
Routing:
- net MX6: track 0.00 -> 43.6 mm
- net N$5: track 0.00 -> 20.1 mm
- net MY0: track 0.00 -> 13.2 mm
- net N$4: track 0.00 -> 8.99 mm
- net N$28: track 0.00 -> 8.49 mm
- net N$14: track 0.00 -> 3.57 mm
- net N$3: track 0.00 -> 3.49 mm
- net N$9: track 0.00 -> 3.36 mm
- net N$8: track 0.00 -> 3.36 mm
- net N$7: track 0.00 -> 3.36 mm
- net N$6: track 0.00 -> 3.36 mm
- net N$13: track 0.00 -> 3.36 mm
- net N$12: track 0.00 -> 3.36 mm
- net N$11: track 0.00 -> 3.36 mm
- net N$10: track 0.00 -> 3.36 mm

Commit message: .
Parts:
- added LED-5, LED-6, LED-7, LED-8, LED-CL, LED-FN: SK6812-E-REVERSE, ts_keyboards:SK6812-E-MILL
- added U$10, U$12, U$13, U$15, U$6, U$9: MOUNTING-HOLE-WIDE, ts_keyboards:MOUNTING-HOLE-WIDE
- added U$14: TVS_SMF9.0CA, ts_keyboards:SOD123FL-BI
- added U$3: ESD_SRV05-4, ts_keyboards:SOT-23-6L
- added U$4: MOUNTING-HOLE, ts_keyboards:MOUNTING-HOLE
- added U$5, U$8: MOUNTING-HOLE-VWIDE, ts_keyboards:MOUNTING-HOLE-VWIDE
- added U$7: PTC_ASMD1206, ts_keyboards:SMD_PTC
- added X1: (no value), ts_keyboards:USB_C_CUSB31-CFM2AX-01-X
- moved D1 18.0 mm to (4.00, 76.0)
- moved D34 4.24 mm to (128.9, 55.0)
- turned S_BSL to 180 degrees
- turned S_FN1 to 180 degrees
Connections:
- new net N$29: LED-5.4-DIN, LED-CL.2-DOUT
- new net N$63: LED-5.2-DOUT, LED-6.4-DIN
- new net N$64: LED-6.2-DOUT, LED-7.4-DIN
- new net N$65: LED-7.2-DOUT, LED-8.4-DIN
- new net N$66: LED-8.2-DOUT, LED-FN.4-DIN
- new net VBUS: X1.A4B9, X1.B4A9
- net GND: now also LED-5.3-GND, LED-6.3-GND, LED-7.3-GND, LED-8.3-GND, LED-CL.3-GND, LED-FN.3-GND, X1.A1B12, X1.B1A12
- net VCC: now also LED-5.1-VDD, LED-6.1-VDD, LED-7.1-VDD, LED-8.1-VDD, LED-CL.1-VDD, LED-FN.1-VDD
Routing:
- net MX6: track 43.6 -> 0.00 mm
- net N$28: track 8.49 -> 0.18 mm

Commit message: .
Parts:
- removed LED-FN: SK6812-E-REVERSE, ts_keyboards:SK6812-E-MILL
- added C1, C2: 0.1uF, SparkFun-Capacitors:0603
- added C3, C4: 0.22uF, SparkFun-Capacitors:0603
- added C5: 1nF, SparkFun-Capacitors:0603
- added IC1: MC74VHC1G50, __untitled:SC-74A
- added IC2: REG1117, burr-brown:SOT223
- added J2: (no value), __untitled:1X04_1MM_RA
- added R1, R2: 1.5k, SparkFun-Resistors:0603
- added R3: 150k, SparkFun-Resistors:0603
- added R4: 75, SparkFun-Resistors:0603
- added S1: Reset, SparkFun-Switches:TACTILE_SWITCH_SMD_5.2MM
- added S2: BOOT, SparkFun-Switches:TACTILE_SWITCH_SMD_5.2MM
- moved X1 1.10 mm to (18.2, 95.5)
- turned S_2 to 0 degrees
Connections:
- new net D+: J2.3, J6.3, U$3.P$3, U$3.P$6, X1.A6, X1.B6
- new net D-: J2.2, J6.5, U$3.P$1, U$3.P$4, X1.A7, X1.B7
- new net LED: IC1.2, J6.47
- new net N$67: R1.1, X1.A5
- new net N$68: IC1.4, LED-CL.4-DIN
- new net N$69: R2.1, X1.B5
- new net N$70: J6.11, S2.3, S2.4
- new net VIN/3: J6.49, R3.1, R4.2
- new net VSUP: C2.1, C4.1, IC2.3, J2.1, R3.2, U$14.P$1, U$7.P$2
- net GND: now also C1.2, C2.2, C3.2, C4.2, C5.2, IC1.5, IC2.1, J2.4, R1.2, R2.2, R4.1, S1.1, S1.2, S2.1, S2.2, U$14.P$2, U$3.P$2; no longer LED-FN.3-GND
- net N$66: now also J6.6, S1.3, S1.4; no longer LED-8.2-DOUT, LED-FN.4-DIN
- net VBUS: now also IC1.3, LED-5.1-VDD, LED-6.1-VDD, LED-7.1-VDD, LED-8.1-VDD, LED-CL.1-VDD, U$3.P$5, U$7.P$1
- net VCC: now also C1.1, C3.1, C5.1, IC2.2, J6.4; no longer LED-5.1-VDD, LED-6.1-VDD, LED-7.1-VDD, LED-8.1-VDD, LED-CL.1-VDD, LED-FN.1-VDD
Routing:
- net N$3: track 3.49 -> 0.59 mm

Commit message: .
Parts:
- removed U$9: MOUNTING-HOLE-WIDE, ts_keyboards:MOUNTING-HOLE-WIDE
Changed lines of the file:
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@@
 <drawing>
 <settings>
-<setting alwaysvectorfont="no"/>
+<setting alwaysvectorfont="yes"/>
 <setting verticaltext="up"/>
 </settings>
@@
 <wire x1="22.7" y1="87" x2="22.7" y2="94" width="0.01" layer="49" style="shortdash"/>
 <circle x="29.15" y="46.6" radius="2.5" width="0.01" layer="49"/>
+<hole x="129.2" y="47.8" drill="2.5"/>
+<hole x="127.2" y="47.8" drill="2.5"/>
 </plain>
 <attributes>
@@
 </element>
 <element name="U$8" library="ts_keyboards" package="MOUNTING-HOLE-VWIDE" value="MOUNTING-HOLE-VWIDE" x="282.5" y="38.3" locked="yes" smashed="yes"/>
-<element name="U$9" library="ts_keyboards" package="MOUNTING-HOLE-WIDE" value="MOUNTING-HOLE-WIDE" x="128.2" y="47.8" locked="yes" smashed="yes"/>
 <element name="U$10" library="ts_keyboards" package="MOUNTING-HOLE-WIDE" value="MOUNTING-HOLE-WIDE" x="74.2" y="16.9" locked="yes" smashed="yes"/>
 <element name="U$12" library="ts_keyboards" package="MOUNTING-HOLE-WIDE" value="MOUNTING-HOLE-WIDE" x="190.5" y="9.6" locked="yes" smashed="yes"/>

Commit message: additional protection & diode placements
Parts:
- added C6: 4.7nf, OPL_Capacitor:C0603
- added D62: 1N4148, adafruit:SOD-123
- added R5: 1M, OPL_Resistor:R0603
- C2: value 0.1uF -> 0.22uF
- C3: value 0.22uF -> 1nF
- C4: value 0.22uF -> 0.1uF
- C5: value 1nF -> 0.22uF
- moved R1 253.2 mm to (28.0, 91.0), turned to 270 degrees
- moved R2 251.3 mm to (31.0, 91.0), turned to 270 degrees
- moved C3 236.2 mm to (38.0, 42.0)
- moved C4 232.3 mm to (42.0, 36.0), turned to 180 degrees
- moved R3 232.1 mm to (42.0, 42.0)
- moved C5 232.0 mm to (42.0, 39.0), turned to 180 degrees
- moved R4 228.0 mm to (46.0, 42.0)
- moved IC1 133.7 mm to (30.0, 54.0)
- moved U$7 105.1 mm to (17.0, 77.0)
- moved U$14 93.5 mm to (25.0, 59.0), turned to 180 degrees
- moved U$3 93.3 mm to (25.0, 75.0), turned to 270 degrees
- moved D18 23.4 mm to (63.0, 59.1), turned to 180 degrees
- moved C1 22.5 mm to (38.0, 36.0), turned to 0 degrees
- moved D34 22.5 mm to (113.0, 39.1), turned to 0 degrees
- moved D29 22.0 mm to (23.0, 38.8), turned to 180 degrees
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Connections:
- new net N$71: C6.2, R5.2, X1.M1, X1.M2, X1.M3, X1.M4
- net D+: now also U$3.P$1; no longer U$3.P$3
- net D-: now also U$3.P$3; no longer U$3.P$1
- net GND: now also C6.1, R5.1
- net VCC: now also C2.1, D62.A; no longer C5.1
- net VSUP: now also C5.1, D62.C; no longer C2.1
Routing:
- net N$5: track 20.1 -> 0.05 mm
- net MY0: track 13.2 -> 0.00 mm
- net N$4: track 8.99 -> 0.05 mm
- net N$14: track 3.57 -> 0.00 mm
- net N$6: track 3.36 -> 6.88 mm
- net N$13: track 3.36 -> 6.88 mm
- net N$9: track 3.36 -> 0.00 mm
- net N$8: track 3.36 -> 0.00 mm
- net N$7: track 3.36 -> 0.00 mm
- net N$12: track 3.36 -> 0.00 mm
- net N$11: track 3.36 -> 0.00 mm
- net N$10: track 3.36 -> 0.00 mm
- net N$3: track 0.59 -> 0.00 mm

Commit message: wip
Parts:
- added J1: (no value), SparkFun-Connectors:1X02
- added J3: JTAG, SparkFun-Connectors:2X5-PTH-1.27MM
- added JP1: OPT, SparkFun-Jumpers:SMT-JUMPER_2_NC_PASTE_NO-SILK
- C6: value 4.7nf -> 4.7nF; device OPL_Capacitor:C0603 -> SparkFun-Capacitors:0603
- IC1: device __untitled:SC-74A -> ts_keyboards:SC-74A
- R4: value 75 -> 75K
- R5: value 1M -> 1000K; device OPL_Resistor:R0603 -> SparkFun-Resistors:0603
- moved R3 19.0 mm to (42.0, 61.0)
- moved R4 16.5 mm to (42.0, 58.0), turned to 180 degrees
- moved D2 12.0 mm to (35.0, 89.0)
- moved IC1 5.00 mm to (25.0, 54.0)
- moved R2 4.47 mm to (27.0, 89.0), turned to 180 degrees
- moved R5 2.24 mm to (11.0, 92.0)
- moved C6 2.00 mm to (11.0, 89.0), turned to 0 degrees
- moved R1 1.41 mm to (27.0, 92.0), turned to 180 degrees
- moved U$7 1.41 mm to (18.0, 78.0), turned to 270 degrees
- turned U$3 to 90 degrees
Connections:
- removed net N$66: J6.6, S1.3, S1.4
- removed net N$70 (its old number): J6.11, S2.3, S2.4
- new net !BOOT: J1.1, J6.11, S2.3, S2.4
- new net !RESET: J3.10, J6.6, S1.3, S1.4
- new net N$68: JP1.1, R3.2
- new net P$1: U$10.P$10, U$10.P$2, U$10.P$3, U$10.P$4, U$10.P$5, U$10.P$7, U$10.P$8, U$10.P$9, U$12.P$10, U$12.P$2, U$12.P$3, U$12.P$4, U$12.P$5, U$12.P$7, U$12.P$8, U$12.P$9, U$13.P$10, U$13.P$2, U$13.P$3, U$13.P$4, U$13.P$5, U$13.P$7, U$13.P$8, U$13.P$9, U$15.P$10, U$15.P$2, U$15.P$3, U$15.P$4, U$15.P$5, U$15.P$7, U$15.P$8, U$15.P$9, U$4.P$10, U$4.P$2, U$4.P$3, U$4.P$7, U$4.P$8, U$4.P$9, U$5.P$1, U$5.P$10, U$5.P$2, U$5.P$3, U$5.P$4, U$5.P$5, U$5.P$6, U$5.P$7, U$5.P$8, U$5.P$9, U$6.P$10, U$6.P$2, U$6.P$3, U$6.P$4, U$6.P$5, U$6.P$7, U$6.P$8, U$6.P$9, U$8.P$1, U$8.P$10, U$8.P$2, U$8.P$3, U$8.P$4, U$8.P$5, U$8.P$6, U$8.P$7, U$8.P$8, U$8.P$9
- new net SWDCK: J3.4, J6.21
- new net SWDIO: J3.2, J6.23
- net GND: now also C6.2, IC1.3, J1.2, J3.3, J3.5, J3.9; no longer C6.1, IC1.5
- net N$71: now also C6.1; no longer C6.2
- net VBUS: no longer IC1.3, LED-5.1-VDD, LED-6.1-VDD, LED-7.1-VDD, LED-8.1-VDD, LED-CL.1-VDD
- net VCC: now also C4.1, C5.1, D62.C, IC2.3, J3.1
- net VSUP: now also IC1.5, JP1.2, LED-5.1-VDD, LED-6.1-VDD, LED-7.1-VDD, LED-8.1-VDD, LED-CL.1-VDD; no longer C4.1, C5.1, D62.C, IC2.3, R3.2
Routing:
- net D+: track 0.00 -> 44.9 mm, vias 0 -> 2
- net D-: track 0.00 -> 36.5 mm, vias 0 -> 2
- net VBUS: track 0.00 -> 30.2 mm, vias 0 -> 2
- net N$69: track 0.00 -> 13.2 mm, vias 0 -> 2
- net N$67: track 0.00 -> 11.9 mm
- net N$71: track 0.00 -> 8.13 mm
- added copper zone on layer 1, net GND
- added copper zone on layer 16, net GND

Commit message: wip
Parts:
- S-EQL, S_0, S_1, S_2, S_3, S_4, S_5, S_6, S_7, S_8, S_9, S_A, S_B, S_BSL, S_BSP, S_C, S_CB, S_COM, S_CPS, S_D, S_DOT, S_E, S_ENT, S_ESC, S_F, S_FN1, S_FSL, S_G, S_H, S_I, S_J, S_K, S_L, S_LAL, S_LCT, S_LGU, S_LSH, S_M, S_MIN, S_N, S_O, S_OB, S_P, S_Q, S_QUO, S_R, S_RAL, S_RCT, S_RGU, S_RSH, S_S, S_SCL, S_SPC, S_T, S_TAB, S_U, S_V, S_W, S_X, S_Y, S_Z: value MX-5-PIN-HOTSWAP -> MX-5-PIN-HOTSWAP-PAD; device ts_keyboards:MX-5-PIN-HOTSWAP -> ts_keyboards:MX-5-PIN-HOTSWAP-PAD
- moved J3 51.7 mm to (95.0, 61.5), flipped to the bottom
- moved D35 21.0 mm to (127.5, 59.6)
- moved D19 19.2 mm to (92.0, 75.9)
- moved D28 18.6 mm to (272.0, 73.1), turned to 0 degrees
- moved D30 12.9 mm to (49.0, 39.1), turned to 0 degrees
- moved D58 12.9 mm to (210.8, 18.0)
- moved D50 12.0 mm to (179.8, 24.9)
- moved D45 11.8 mm to (84.8, 24.5)
- moved D12 9.49 mm to (225.0, 77.0)
- moved D53 7.47 mm to (253.4, 25.1)
- moved D55 5.73 mm to (30.2, 17.9)
- moved D31 5.02 mm to (56.5, 44.1)
- moved D32 5.02 mm to (75.5, 44.1)
- moved D33 5.02 mm to (94.5, 44.1)
- moved D34 5.02 mm to (113.5, 44.1)
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- renumbered U$10 to SA1, U$12 to SG3, U$13 to SA3, U$15 to SA2, U$4 to SC1, U$5 to SG1, U$6 to SC2, U$8 to SG4
Connections:
- removed net P$1: SA1.P$10, SA1.P$2, SA1.P$3, SA1.P$4, SA1.P$5, SA1.P$7, SA1.P$8, SA1.P$9, SA2.P$10, SA2.P$2, SA2.P$3, SA2.P$4, SA2.P$5, SA2.P$7, SA2.P$8, SA2.P$9, SA3.P$10, SA3.P$2, SA3.P$3, SA3.P$4, SA3.P$5, SA3.P$7, SA3.P$8, SA3.P$9, SC1.P$10, SC1.P$2, SC1.P$3, SC1.P$7, SC1.P$8, SC1.P$9, SC2.P$10, SC2.P$2, SC2.P$3, SC2.P$4, SC2.P$5, SC2.P$7, SC2.P$8, SC2.P$9, SG1.P$1, SG1.P$10, SG1.P$2, SG1.P$3, SG1.P$4, SG1.P$5, SG1.P$6, SG1.P$7, SG1.P$8, SG1.P$9, SG3.P$10, SG3.P$2, SG3.P$3, SG3.P$4, SG3.P$5, SG3.P$7, SG3.P$8, SG3.P$9, SG4.P$1, SG4.P$10, SG4.P$2, SG4.P$3, SG4.P$4, SG4.P$5, SG4.P$6, SG4.P$7, SG4.P$8, SG4.P$9
- new net SA1: SA1.P$10, SA1.P$2, SA1.P$3, SA1.P$4, SA1.P$5, SA1.P$7, SA1.P$8, SA1.P$9
- new net SA2: SA2.P$10, SA2.P$2, SA2.P$3, SA2.P$4, SA2.P$5, SA2.P$7, SA2.P$8, SA2.P$9
- new net SA3: SA3.P$10, SA3.P$2, SA3.P$3, SA3.P$4, SA3.P$5, SA3.P$7, SA3.P$8, SA3.P$9
- new net SC1: SC1.P$10, SC1.P$2, SC1.P$3, SC1.P$7, SC1.P$8, SC1.P$9
- new net SC2: SC2.P$10, SC2.P$2, SC2.P$3, SC2.P$4, SC2.P$5, SC2.P$7, SC2.P$8, SC2.P$9
- new net SG1: SG1.P$1, SG1.P$10, SG1.P$2, SG1.P$3, SG1.P$4, SG1.P$5, SG1.P$6, SG1.P$7, SG1.P$8, SG1.P$9
- new net SG3: SG3.P$10, SG3.P$2, SG3.P$3, SG3.P$4, SG3.P$5, SG3.P$7, SG3.P$8, SG3.P$9
- new net SG4: SG4.P$1, SG4.P$10, SG4.P$2, SG4.P$3, SG4.P$4, SG4.P$5, SG4.P$6, SG4.P$7, SG4.P$8, SG4.P$9
- net MY0: now also S_1.P$4, S_2.P$4, S_3.P$4, S_4.P$4, S_5.P$4, S_6.P$4, S_7.P$4, S_ESC.P$4
- net MY1: now also S_E.P$4, S_Q.P$4, S_R.P$4, S_T.P$4, S_TAB.P$4, S_U.P$4, S_W.P$4, S_Y.P$4
- net MY2: now also S_A.P$4, S_CPS.P$4, S_D.P$4, S_F.P$4, S_G.P$4, S_H.P$4, S_J.P$4, S_S.P$4
- net MY3: now also S_B.P$4, S_C.P$4, S_LSH.P$4, S_N.P$4, S_V.P$4, S_X.P$4, S_Z.P$4
- net MY4: now also S_FN1.P$4, S_LAL.P$4, S_LCT.P$4, S_LGU.P$4, S_RAL.P$4, S_RCT.P$4, S_RGU.P$4, S_SPC.P$4
- net MY5: now also S-EQL.P$4, S_0.P$4, S_8.P$4, S_9.P$4, S_BSP.P$4, S_MIN.P$4
- net MY6: now also S_BSL.P$4, S_CB.P$4, S_I.P$4, S_O.P$4, S_OB.P$4, S_P.P$4
- net MY7: now also S_ENT.P$4, S_K.P$4, S_L.P$4, S_QUO.P$4, S_SCL.P$4
- net MY8: now also S_COM.P$4, S_DOT.P$4, S_FSL.P$4, S_M.P$4, S_RSH.P$4
- net N$1: now also S_ESC.P$3
- net N$10: now also S_9.P$3
- net N$11: now also S_0.P$3
- net N$12: now also S_MIN.P$3
- net N$13: now also S-EQL.P$3
- net N$14: now also S_BSP.P$3
- net N$15: now also S_TAB.P$3
- net N$16: now also S_Q.P$3
- net N$17: now also S_W.P$3
- net N$18: now also S_E.P$3
- net N$19: now also S_R.P$3
- net N$2: now also S_1.P$3
- net N$20: now also S_T.P$3
- net N$21: now also S_Y.P$3
- net N$22: now also S_U.P$3
- net N$23: now also S_I.P$3
- net N$24: now also S_O.P$3
- net N$25: now also S_P.P$3
- net N$26: now also S_OB.P$3
- net N$27: now also S_CB.P$3
- net N$28: now also S_BSL.P$3
- net N$3: now also S_2.P$3
- net N$30: now also S_A.P$3
- net N$31: now also S_S.P$3
- net N$32: now also S_D.P$3
- net N$33: now also S_F.P$3
- net N$34: now also S_G.P$3
- net N$35: now also S_H.P$3
- net N$36: now also S_J.P$3
- net N$37: now also S_K.P$3
- net N$38: now also S_L.P$3
- net N$39: now also S_SCL.P$3
- net N$4: now also S_3.P$3
- net N$40: now also S_QUO.P$3
- net N$41: now also S_ENT.P$3
- net N$42: now also S_LSH.P$3
- net N$43: now also S_Z.P$3
- net N$44: now also S_X.P$3
- net N$45: now also S_C.P$3
- net N$46: now also S_V.P$3
- net N$47: now also S_B.P$3
- net N$48: now also S_N.P$3
- net N$49: now also S_M.P$3
- net N$5: now also S_4.P$3
- net N$50: now also S_COM.P$3
- net N$51: now also S_DOT.P$3
- net N$52: now also S_FSL.P$3
- net N$53: now also S_RSH.P$3
- net N$54: now also S_LCT.P$3
- net N$55: now also S_LGU.P$3
- net N$56: now also S_LAL.P$3
- net N$57: now also S_SPC.P$3
- net N$58: now also S_FN1.P$3
- net N$59: now also S_RAL.P$3
- net N$6: now also S_5.P$3
- net N$60: now also S_RGU.P$3
- net N$61: now also S_RCT.P$3
- net N$62: now also S_CPS.P$3
- net N$7: now also S_6.P$3
- net N$8: now also S_7.P$3
- net N$9: now also S_8.P$3
- net VCC: no longer C4.1, C5.1, D62.C, IC2.3
- net VSUP: now also C4.1, C5.1, D62.C, IC2.3
Routing:
- net VSUP: track 0.00 -> 373.0 mm, vias 0 -> 7
- net MX3: track 0.00 -> 291.1 mm, vias 0 -> 3
- net MY4: track 0.00 -> 282.7 mm, vias 0 -> 1
- net MY2: track 0.00 -> 223.7 mm, vias 0 -> 8
- net MX7: track 0.00 -> 216.0 mm, vias 0 -> 4
- net MX2: track 0.00 -> 204.9 mm, vias 0 -> 5
- net MX0: track 0.00 -> 180.2 mm, vias 0 -> 3
- net MX4: track 0.00 -> 173.2 mm, vias 0 -> 5
- net MX1: track 0.00 -> 166.5 mm, vias 0 -> 6
- net MY1: track 0.00 -> 162.7 mm, vias 0 -> 8
- net MX5: track 0.00 -> 159.5 mm, vias 0 -> 6
- net MY0: track 0.00 -> 154.5 mm
- net MX6: track 0.00 -> 138.0 mm
- net MY6: track 0.00 -> 120.5 mm, vias 0 -> 7
- net MY7: track 0.00 -> 109.6 mm, vias 0 -> 6
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Other:
- board text added: "AP2"
- board text added: "BOOT"
- board text added: "CMN"
- board text added: "GH60"
- board text added: "JTAG"
- board text added: "RESET"
