File: EAGLE/vr61/vr60.sch (EAGLE design)
At the start: 188 parts

Commit message: .
Parts:
- removed S1, S10, S11, S12, S13, S14, S15, S16, S17, S18, S19, S2, S20, S21, S22, S23, S24, S25, S26, S27, S28, S29, S3, S30, S31, S32, S33, S34, S35, S36, S37, S38, S39, S4, S40, S41, S42, S43, S44, S45, S46, S47, S48, S49, S5, S50, S51, S52, S53, S54, S55, S56, S57, S58, S59, S6, S60, S61, S7, S8, S9: MX-5-PIN-HOTSWAP, ts_keyboards:MX-5-PIN-HOTSWAP
- added H5: STAND-OFF-REFLOW2.5MM_TALL, SparkFun-Hardware:STAND-OFF-REFLOW2.5MM_TALL
- added J6: MICROMOD-2222-C, SparkFun-MicroMod:MICROMOD-2222-C
- added S-EQL, S_0, S_1, S_2, S_3, S_4, S_5, S_6, S_7, S_8, S_9, S_A, S_B, S_BSL, S_BSP, S_C, S_CB, S_COM, S_CPS, S_D, S_DOT, S_E, S_ENT, S_ESC, S_F, S_FN1, S_FSL, S_G, S_H, S_I, S_J, S_K, S_L, S_LAL, S_LCT, S_LGU, S_LSH, S_M, S_MIN, S_N, S_O, S_OB, S_P, S_Q, S_QUO, S_R, S_RAL, S_RCT, S_RGU, S_RSH, S_S, S_SCL, S_SPC, S_T, S_TAB, S_U, S_V, S_W, S_X, S_Y, S_Z: MX-5-PIN-HOTSWAP, ts_keyboards:MX-5-PIN-HOTSWAP
Connections:
- removed net COL10: D11.C, D25.C, D39.C, D51.C, D58.C
- removed net COL11: D12.C, D26.C, D40.C, D52.C, D59.C
- removed net COL12: D13.C, D27.C, D60.C
- removed net COL13: D14.C, D28.C, D41.C, D53.C, D61.C
- removed net COL8: D23.C, D37.C, D49.C, D9.C
- removed net COL9: D10.C, D24.C, D38.C, D50.C
- removed net N$29: D29.A, S29.P
- new net GND: H5.1
- new net N$62: D29.A, S_CPS.P
- new net ROW5: S-EQL.S, S_0.S, S_8.S, S_9.S, S_BSP.S, S_MIN.S
- new net ROW6: S_BSL.S, S_CB.S, S_I.S, S_O.S, S_OB.S, S_P.S
- new net ROW7: S_ENT.S, S_K.S, S_L.S, S_QUO.S, S_SCL.S
- new net ROW8: S_COM.S, S_DOT.S, S_FSL.S, S_M.S, S_RSH.S
- net COL0: now also D23.C, D37.C, D49.C, D9.C
- net COL1: now also D10.C, D24.C, D38.C, D50.C
- net COL2: now also D11.C, D25.C, D39.C, D51.C
- net COL3: now also D12.C, D26.C, D40.C, D52.C, D57.C
- net COL4: now also D13.C, D27.C, D58.C
- net COL5: now also D53.C, D59.C
- net COL6: now also D14.C, D28.C, D41.C, D60.C; no longer D57.C
- net COL7: now also D61.C
- net N$1: now also S_ESC.P; no longer S1.P
- net N$10: now also S_9.P; no longer S10.P
- net N$11: now also S_0.P; no longer S11.P
- net N$12: now also S_MIN.P; no longer S12.P
- net N$13: now also S-EQL.P; no longer S13.P
- net N$14: now also S_BSP.P; no longer S14.P
- net N$15: now also S_TAB.P; no longer S15.P
- net N$16: now also S_Q.P; no longer S16.P
- net N$17: now also S_W.P; no longer S17.P
- net N$18: now also S_E.P; no longer S18.P
- net N$19: now also S_R.P; no longer S19.P
- net N$2: now also S_1.P; no longer S2.P
- net N$20: now also S_T.P; no longer S20.P
- net N$21: now also S_Y.P; no longer S21.P
- net N$22: now also S_U.P; no longer S22.P
- net N$23: now also S_I.P; no longer S23.P
- net N$24: now also S_O.P; no longer S24.P
- net N$25: now also S_P.P; no longer S25.P
- net N$26: now also S_OB.P; no longer S26.P
- net N$27: now also S_CB.P; no longer S27.P
- net N$28: now also S_BSL.P; no longer S28.P
- net N$3: now also S_2.P; no longer S3.P
- net N$30: now also S_A.P; no longer S30.P
- net N$31: now also S_S.P; no longer S31.P
- net N$32: now also S_D.P; no longer S32.P
- net N$33: now also S_F.P; no longer S33.P
- net N$34: now also S_G.P; no longer S34.P
- net N$35: now also S_H.P; no longer S35.P
- net N$36: now also S_J.P; no longer S36.P
- net N$37: now also S_K.P; no longer S37.P
- net N$38: now also S_L.P; no longer S38.P
- net N$39: now also S_SCL.P; no longer S39.P
- net N$4: now also S_3.P; no longer S4.P
- net N$40: now also S_QUO.P; no longer S40.P
- net N$41: now also S_ENT.P; no longer S41.P
- net N$42: now also S_LSH.P; no longer S42.P
- net N$43: now also S_Z.P; no longer S43.P
- net N$44: now also S_X.P; no longer S44.P
- net N$45: now also S_C.P; no longer S45.P
- net N$46: now also S_V.P; no longer S46.P
- net N$47: now also S_B.P; no longer S47.P
- net N$48: now also S_N.P; no longer S48.P
- net N$49: now also S_M.P; no longer S49.P
- net N$5: now also S_4.P; no longer S5.P
- net N$50: now also S_COM.P; no longer S50.P
- net N$51: now also S_DOT.P; no longer S51.P
- net N$52: now also S_FSL.P; no longer S52.P
- net N$53: now also S_RSH.P; no longer S53.P
- net N$54: now also S_LCT.P; no longer S54.P
- net N$55: now also S_LGU.P; no longer S55.P
- net N$56: now also S_LAL.P; no longer S56.P
- net N$57: now also S_SPC.P; no longer S57.P
- net N$58: now also S_FN1.P; no longer S58.P
- net N$59: now also S_RAL.P; no longer S59.P
- net N$6: now also S_5.P; no longer S6.P
- net N$60: now also S_RGU.P; no longer S60.P
- net N$61: now also S_RCT.P; no longer S61.P
- net N$7: now also S_6.P; no longer S7.P
- net N$8: now also S_7.P; no longer S8.P
- net N$9: now also S_8.P; no longer S9.P
- net ROW0: now also S_1.S, S_2.S, S_3.S, S_4.S, S_5.S, S_6.S, S_7.S, S_ESC.S; no longer S1.S, S10.S, S11.S, S12.S, S13.S, S14.S, S2.S, S3.S, S4.S, S5.S, S6.S, S7.S, S8.S, S9.S
- net ROW1: now also S_E.S, S_Q.S, S_R.S, S_T.S, S_TAB.S, S_U.S, S_W.S, S_Y.S; no longer S15.S, S16.S, S17.S, S18.S, S19.S, S20.S, S21.S, S22.S, S23.S, S24.S, S25.S, S26.S, S27.S, S28.S
- net ROW2: now also S_A.S, S_CPS.S, S_D.S, S_F.S, S_G.S, S_H.S, S_J.S, S_S.S; no longer S29.S, S30.S, S31.S, S32.S, S33.S, S34.S, S35.S, S36.S, S37.S, S38.S, S39.S, S40.S, S41.S
- net ROW3: now also S_B.S, S_C.S, S_LSH.S, S_N.S, S_V.S, S_X.S, S_Z.S; no longer S42.S, S43.S, S44.S, S45.S, S46.S, S47.S, S48.S, S49.S, S50.S, S51.S, S52.S, S53.S
- net ROW4: now also S_FN1.S, S_LAL.S, S_LCT.S, S_LGU.S, S_RAL.S, S_RCT.S, S_RGU.S, S_SPC.S; no longer S54.S, S55.S, S56.S, S57.S, S58.S, S59.S, S60.S, S61.S

Commit message: .
Connections:
- removed net COL0: D1.C, D15.C, D23.C, D29.C, D37.C, D42.C, D49.C, D54.C, D9.C
- removed net COL1: D10.C, D16.C, D2.C, D24.C, D30.C, D38.C, D50.C, D55.C
- removed net COL2: D11.C, D17.C, D25.C, D3.C, D31.C, D39.C, D43.C, D51.C, D56.C
- removed net COL3: D12.C, D18.C, D26.C, D32.C, D4.C, D40.C, D44.C, D52.C, D57.C
- removed net COL4: D13.C, D19.C, D27.C, D33.C, D45.C, D5.C, D58.C
- removed net COL5: D20.C, D34.C, D46.C, D53.C, D59.C, D6.C
- removed net COL6: D14.C, D21.C, D28.C, D35.C, D41.C, D47.C, D60.C, D7.C
- removed net COL7: D22.C, D36.C, D48.C, D61.C, D8.C
- removed net ROW0: S_1.S, S_2.S, S_3.S, S_4.S, S_5.S, S_6.S, S_7.S, S_ESC.S
- removed net ROW1: S_E.S, S_Q.S, S_R.S, S_T.S, S_TAB.S, S_U.S, S_W.S, S_Y.S
- removed net ROW2: S_A.S, S_CPS.S, S_D.S, S_F.S, S_G.S, S_H.S, S_J.S, S_S.S
- removed net ROW3: S_B.S, S_C.S, S_LSH.S, S_N.S, S_V.S, S_X.S, S_Z.S
- removed net ROW4: S_FN1.S, S_LAL.S, S_LCT.S, S_LGU.S, S_RAL.S, S_RCT.S, S_RGU.S, S_SPC.S
- removed net ROW5: S-EQL.S, S_0.S, S_8.S, S_9.S, S_BSP.S, S_MIN.S
- removed net ROW6: S_BSL.S, S_CB.S, S_I.S, S_O.S, S_OB.S, S_P.S
- removed net ROW7: S_ENT.S, S_K.S, S_L.S, S_QUO.S, S_SCL.S
- removed net ROW8: S_COM.S, S_DOT.S, S_FSL.S, S_M.S, S_RSH.S
- new net MX0: D1.C, D15.C, D23.C, D29.C, D37.C, D42.C, D49.C, D54.C, D9.C, J6.D1/CAM_TRIG
- new net MX1: D10.C, D16.C, D2.C, D24.C, D30.C, D38.C, D50.C, D55.C, J6.I2C_!INT!
- new net MX2: D11.C, D17.C, D25.C, D3.C, D31.C, D39.C, D43.C, D51.C, D56.C, J6.I2C_SCL
- new net MX3: D12.C, D18.C, D26.C, D32.C, D4.C, D40.C, D44.C, D52.C, D57.C, J6.A1
- new net MX4: D13.C, D19.C, D27.C, D33.C, D45.C, D5.C, D58.C, J6.I2C_SDA
- new net MX5: D20.C, D34.C, D46.C, D53.C, D59.C, D6.C, J6.D0
- new net MX6: D14.C, D21.C, D28.C, D35.C, D41.C, D47.C, D60.C, D7.C, J6.TX1
- new net MX7: D22.C, D36.C, D48.C, D61.C, D8.C, J6.RX1
- new net MY0: J6.AUD_OUT/CAM_MCLK, S_1.S, S_2.S, S_3.S, S_4.S, S_5.S, S_6.S, S_7.S, S_ESC.S
- new net MY1: J6.AUD_IN/CAM_PCLK, S_E.S, S_Q.S, S_R.S, S_T.S, S_TAB.S, S_U.S, S_W.S, S_Y.S
- new net MY2: J6.AUD_LRCLK, S_A.S, S_CPS.S, S_D.S, S_F.S, S_G.S, S_H.S, S_J.S, S_S.S
- new net MY3: J6.AUD_BCLK, S_B.S, S_C.S, S_LSH.S, S_N.S, S_V.S, S_X.S, S_Z.S
- new net MY4: J6.G4/BUS4, S_FN1.S, S_LAL.S, S_LCT.S, S_LGU.S, S_RAL.S, S_RCT.S, S_RGU.S, S_SPC.S
- new net MY5: J6.G3/BUS3, S-EQL.S, S_0.S, S_8.S, S_9.S, S_BSP.S, S_MIN.S
- new net MY6: J6.G2/BUS2, S_BSL.S, S_CB.S, S_I.S, S_O.S, S_OB.S, S_P.S
- new net MY7: J6.G1/BUS1, S_ENT.S, S_K.S, S_L.S, S_QUO.S, S_SCL.S
- new net MY8: J6.G0/BUS0, S_COM.S, S_DOT.S, S_FSL.S, S_M.S, S_RSH.S
- new net VCC: J6.3.3V
- net GND: now also J6.GND

Commit message: .
Parts:
- added LED-5, LED-6, LED-7, LED-8, LED-CL, LED-FN: SK6812-E-REVERSE, ts_keyboards:SK6812-E-REVERSE
- added U$10, U$12, U$13, U$15, U$6, U$9: MOUNTING-HOLE-WIDE, ts_keyboards:MOUNTING-HOLE-WIDE
- added U$14: TVS_SMF9.0CA, ts_keyboards:TVS_SMF9.0CA
- added U$3: ESD_SRV05-4, ts_keyboards:ESD_SRV05-4
- added U$4: MOUNTING-HOLE, ts_keyboards:MOUNTING-HOLE
- added U$5, U$8: MOUNTING-HOLE-VWIDE, ts_keyboards:MOUNTING-HOLE-VWIDE
- added U$7: PTC_ASMD1206, ts_keyboards:PTC_ASMD1206
- added X1: (no value), ts_keyboards:USB_C
Connections:
- new net N$29: LED-5.4_DIN, LED-CL.2_DOUT
- new net N$63: LED-5.2_DOUT, LED-6.4_DIN
- new net N$64: LED-6.2_DOUT, LED-7.4_DIN
- new net N$65: LED-7.2_DOUT, LED-8.4_DIN
- new net N$66: LED-8.2_DOUT, LED-FN.4_DIN
- net GND: now also LED-5.3_GND, LED-6.3_GND, LED-7.3_GND, LED-8.3_GND, LED-CL.3_GND, LED-FN.3_GND
- net VCC: now also LED-5.1_VDD, LED-6.1_VDD, LED-7.1_VDD, LED-8.1_VDD, LED-CL.1_VDD, LED-FN.1_VDD

Commit message: .
Parts:
- removed LED-FN: SK6812-E-REVERSE, ts_keyboards:SK6812-E-REVERSE
- added C1, C2: 0.1uF, SparkFun-Capacitors:0.1UF-0603-25V-5%
- added C3, C4: 0.22uF, SparkFun-Capacitors:0.22UF-0603-25V-10%
- added C5: 1nF, SparkFun-Capacitors:1.0NF/1000PF-0603-50V-10%
- added IC1: MC74VHC1G50, __untitled:MC74VHC1G50
- added IC2: REG1117, burr-brown:REG1117
- added J2: (no value), __untitled:C3_UNIFIEDJS-1MM
- added R1, R2: 1.5k, SparkFun-Resistors:1.5KOHM-0603-1/10W-1%
- added R3: 150k, SparkFun-Resistors:150KOHM-0603-1/10W-1%
- added R4: 75, SparkFun-Resistors:75KOHM-0603-1/10W-1%
- added S1: Reset, SparkFun-Switches:MOMENTARY-SWITCH-SPST-SMD-5.2-TALL-REDUNDANT
- added S2: BOOT, SparkFun-Switches:MOMENTARY-SWITCH-SPST-SMD-5.2-TALL-REDUNDANT
Connections:
- new net D+: J2.D+, J6.USB_D+, U$3.P$3, U$3.P$6, X1.D+
- new net D-: J2.D-, J6.USB_D-, U$3.P$1, U$3.P$4, X1.D-
- new net LED: IC1.A, J6.PWM1
- new net N$67: R1.1, X1.CC1
- new net N$68: IC1.Y, LED-CL.4_DIN
- new net N$69: R2.1, X1.CC2
- new net N$70: J6.!BOOT!, S2.2
- new net VBUS: IC1.GND, LED-5.1_VDD, LED-6.1_VDD, LED-7.1_VDD, LED-8.1_VDD, LED-CL.1_VDD, U$3.P$5, U$7.1, X1.VBUS
- new net VIN/3: J6.BATT_VIN/3, R3.1, R4.2
- new net VSUP: C2.1, C4.1, IC2.VIN, J2.VCC, R3.2, U$14.1, U$7.2
- net GND: now also C1.2, C2.2, C3.2, C4.2, C5.2, IC1.VCC, IC2.GND, J2.GND, R1.2, R2.2, R4.1, S1.1, S2.1, U$14.2, U$3.P$2, X1.GND; no longer LED-FN.3_GND
- net N$66: now also J6.!RESET!, S1.2; no longer LED-8.2_DOUT, LED-FN.4_DIN
- net VCC: now also C1.1, C3.1, C5.1, IC2.VOUT, J6.3.3V_EN; no longer LED-5.1_VDD, LED-6.1_VDD, LED-7.1_VDD, LED-8.1_VDD, LED-CL.1_VDD, LED-FN.1_VDD
Other:
- note added: "ESD"
- note added: "OVR-A"
- note added: "OVR-V"
- moved on the sheet: H5, J6, U$14, U$7, X1

Commit message: .
Parts:
- removed U$9: MOUNTING-HOLE-WIDE, ts_keyboards:MOUNTING-HOLE-WIDE
Changed lines of the file:
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@@
 <part name="GND3" library="ts_custom_nick_nacks" deviceset="GND" device=""/>
 <part name="U$8" library="ts_keyboards" deviceset="MOUNTING-HOLE-VWIDE" device=""/>
-<part name="U$9" library="ts_keyboards" deviceset="MOUNTING-HOLE-WIDE" device=""/>
 <part name="U$10" library="ts_keyboards" deviceset="MOUNTING-HOLE-WIDE" device=""/>
 <part name="U$12" library="ts_keyboards" deviceset="MOUNTING-HOLE-WIDE" device=""/>
@@
 </instance>
 <instance part="U$8" gate="G$1" x="266.7" y="25.4" smashed="yes"/>
-<instance part="U$9" gate="G$1" x="266.7" y="30.48" smashed="yes"/>
 <instance part="U$10" gate="G$1" x="264.16" y="30.48" smashed="yes"/>
 <instance part="U$12" gate="G$1" x="259.08" y="30.48" smashed="yes"/>

Commit message: additional protection & diode placements
Parts:
- added C6: 4.7nf, OPL_Capacitor:CERAMIC-4.7NF-50V-10%-X7R(0603)
- added D62: 1N4148, adafruit:DIODESOD-123
- added R5: 1M, OPL_Resistor:SMD-RES-1M-1%-1/10W(0603)
- C2: value 0.1uF -> 0.22uF; device SparkFun-Capacitors:0.1UF-0603-25V-5% -> SparkFun-Capacitors:0.22UF-0603-25V-10%
- C3: value 0.22uF -> 1nF; device SparkFun-Capacitors:0.22UF-0603-25V-10% -> SparkFun-Capacitors:1.0NF/1000PF-0603-50V-10%
- C4: value 0.22uF -> 0.1uF; device SparkFun-Capacitors:0.22UF-0603-25V-10% -> SparkFun-Capacitors:0.1UF-0603-25V-5%
- C5: value 1nF -> 0.22uF; device SparkFun-Capacitors:1.0NF/1000PF-0603-50V-10% -> SparkFun-Capacitors:0.22UF-0603-25V-10%
Connections:
- new net N$71: C6.2, R5.2, X1.SHIELD
- net D+: now also U$3.P$1; no longer U$3.P$3
- net D-: now also U$3.P$3; no longer U$3.P$1
- net GND: now also C6.1, R5.1
- net VCC: now also C2.1, D62.A; no longer C5.1
- net VSUP: now also C5.1, D62.C; no longer C2.1
Other:
- note added: "3V3 Power Supply"
- note added: "ESD and POWER Protection"
- note added: "Micromod Voltage Sensor"
- note added: "RGB LEDs"
- note added: "Sparkfun Micromod Connector"
- note added: "USB-C Port"
- note added: "Unified Daughter Board Connector"
- moved on the sheet: C2, C3, C4, C5, R3, R4

Commit message: wip
Parts:
- added J1: (no value), SparkFun-Connectors:CONN_02
- added J3: JTAG, SparkFun-Connectors:CORTEX_JTAG_DEBUG_MINIMUM_PTH
- added JP1: OPT, SparkFun-Jumpers:JUMPER-SMT_2_NC_PASTE_NO-SILK
- C6: value 4.7nf -> 4.7nF; device OPL_Capacitor:CERAMIC-4.7NF-50V-10%-X7R(0603) -> SparkFun-Capacitors:0.1UF-0603-25V-5%
- IC1: device __untitled:MC74VHC1G50 -> ts_keyboards:MC74VHC1G50
- R4: value 75 -> 75K
- R5: value 1M -> 1000K; device OPL_Resistor:SMD-RES-1M-1%-1/10W(0603) -> SparkFun-Resistors:75KOHM-0603-1/10W-1%
Connections:
- removed net N$66: J6.!RESET!, S1.2
- new net !BOOT: J1.1, J6.!BOOT!, S2.2
- new net !RESET: J3.!RESET, J6.!RESET!, S1.2
- new net SWDCK: J3.SWDCLK, J6.SWDCK
- new net SWDIO: J3.SWDIO, J6.SWDIO
- net GND: now also C6.2, IC1.3_GND, J1.2, J3.GND; no longer C6.1, IC1.VCC
- net LED: now also IC1.A_DIN; no longer IC1.A
- net N$68: now also JP1.1, R3.2; no longer IC1.Y, LED-CL.4_DIN
- net N$70: now also IC1.Y_DOUT, LED-CL.4_DIN; no longer J6.!BOOT!, S2.2
- net N$71: now also C6.1; no longer C6.2
- net VBUS: no longer IC1.GND, LED-5.1_VDD, LED-6.1_VDD, LED-7.1_VDD, LED-8.1_VDD, LED-CL.1_VDD
- net VCC: now also C4.1, C5.1, D62.C, IC2.VIN, J3.VCC
- net VSUP: now also IC1.5_VCC, JP1.2, LED-5.1_VDD, LED-6.1_VDD, LED-7.1_VDD, LED-8.1_VDD, LED-CL.1_VDD; no longer C4.1, C5.1, D62.C, IC2.VIN, R3.2
Other:
- note added: "(Optional) Unified Daughter Board Connector"
- note added: "SHIELD NOISE ISOLATION"
- note removed: "Unified Daughter Board Connector"
- moved on the sheet: H5, LED-5, LED-6, LED-7, LED-8, LED-CL, R3, R4, S1

Commit message: wip
Parts:
- removed U$10, U$12, U$13, U$15, U$6: MOUNTING-HOLE-WIDE, ts_keyboards:MOUNTING-HOLE-WIDE
- removed U$4: MOUNTING-HOLE, ts_keyboards:MOUNTING-HOLE
- removed U$5, U$8: MOUNTING-HOLE-VWIDE, ts_keyboards:MOUNTING-HOLE-VWIDE
- added SA1, SA2, SA3, SC2, SG3: MOUNTING-HOLE-WIDE, ts_keyboards:MOUNTING-HOLE-WIDE
- added SC1: MOUNTING-HOLE, ts_keyboards:MOUNTING-HOLE
- added SG1, SG4: MOUNTING-HOLE-VWIDE, ts_keyboards:MOUNTING-HOLE-VWIDE
- S-EQL, S_0, S_1, S_2, S_3, S_4, S_5, S_6, S_7, S_8, S_9, S_A, S_B, S_BSL, S_BSP, S_C, S_CB, S_COM, S_CPS, S_D, S_DOT, S_E, S_ENT, S_ESC, S_F, S_FN1, S_FSL, S_G, S_H, S_I, S_J, S_K, S_L, S_LAL, S_LCT, S_LGU, S_LSH, S_M, S_MIN, S_N, S_O, S_OB, S_P, S_Q, S_QUO, S_R, S_RAL, S_RCT, S_RGU, S_RSH, S_S, S_SCL, S_SPC, S_T, S_TAB, S_U, S_V, S_W, S_X, S_Y, S_Z: value MX-5-PIN-HOTSWAP -> MX-5-PIN-HOTSWAP-PAD; device ts_keyboards:MX-5-PIN-HOTSWAP -> ts_keyboards:MX-5-PIN-HOTSWAP-PAD
Connections:
- new net SA1: SA1.P$1
- new net SA2: SA2.P$1
- new net SA3: SA3.P$1
- new net SC1: SC1.P$1
- new net SC2: SC2.P$1
- new net SG1: SG1.P$1
- new net SG3: SG3.P$1
- new net SG4: SG4.P$1
- net VCC: no longer C4.1, C5.1, D62.C, IC2.VIN
- net VSUP: now also C4.1, C5.1, D62.C, IC2.VIN
Other:
- moved on the sheet: J3
