File: EAGLE/vr61/vr61-revB.brd (EAGLE design)
At the start: 283 x 93 mm, 244 parts, among them J2 SM04B-SRSS-TB(LF)(SN), J6 MICROMOD-2222-C, Y1 74AHCT1G125

Commit message: wip 2022-07-21
Parts:
- added C12: 1mF, rcl:C0603
- added C13: 100nF, rcl:C0603
- added R7: 470, rcl:R0603
- added R8: 5.1K, rcl:R0603
- added W1: M25C, __untitled:8-SOIC
- moved D29 23.3 mm to (6.00, 58.2)
- renumbered J6 to X1
Connections:
- removed net N$70: LED-CL.4-DIN, Y1.4
- new net EE_CS: W1.1, X1.55
- new net MISO: W1.2, X1.61
- new net MOSI: W1.5, X1.59
- new net N$66: R7.2, Y1.4
- new net N$67: LED-CL.4-DIN, R7.1
- new net SCK: R8.2, W1.6, X1.57
- net GND: now also C12.2, C13.2, R8.1, W1.4
- net VCC: now also C13.1, W1.3, W1.7, W1.8
- net VSUP: now also C12.1
Routing:
- net VCC: track 122.7 -> 169.0 mm, vias 5 -> 8
- net SCK: track 0.00 -> 33.8 mm, vias 0 -> 2
- net MOSI: track 0.00 -> 31.3 mm, vias 0 -> 2
- net MISO: track 0.00 -> 25.5 mm, vias 0 -> 2
- net EE_CS: track 0.00 -> 24.0 mm, vias 0 -> 2
- net N$62: track 18.2 -> 0.09 mm
- net MX3: track 342.4 -> 326.3 mm, vias 6 -> 7
- net MX0: track 311.9 -> 298.4 mm
- net N$70: track 12.3 -> 0.00 mm
- net MY8: track 213.8 -> 209.9 mm
- net MY3: track 173.3 -> 169.8 mm
- net N$32: track 6.01 -> 9.04 mm
- net MY5: track 163.8 -> 161.8 mm
- net MY6: track 233.3 -> 231.3 mm
- net MY7: track 207.1 -> 205.1 mm
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
Commit message: wip 2022-07-21
Parts:
- removed B14, B41, B42, B53: MX-STABS-200U, ts_keyboards:MX-STABS-200U
- removed B57: MX-STABS-625U, ts_keyboards:MX-STABS-625U
- removed S_BSL, S_BSP, S_CB, S_CPS, S_FSL, S_LAL, S_LCT, S_LGU, S_LSH, S_MIN, S_OB, S_QUO, S_RAL, S_RCT, S_RGU, S_RSH, S_SCL: MX-5-PIN-HOTSWAP-PAD, ts_keyboards:MX-5-PIN-HOTSWAP-PAD
- removed Y1: 74AHCT1G125, ts_keyboards:SOT-23-5
- removed Z1, Z10, Z11, Z12, Z13, Z16, Z17, Z18, Z19, Z2, Z20, Z21, Z22, Z23, Z24, Z25, Z26, Z27, Z3, Z30, Z31, Z32, Z33, Z34, Z35, Z36, Z37, Z38, Z39, Z4, Z40, Z43, Z44, Z45, Z46, Z47, Z48, Z49, Z5, Z50, Z51, Z52, Z6, Z7, Z8, Z9: MX-FPRINT-100U19, ts_keyboards:MX-FPRINT-1900-100U
- removed Z14: MX-FPRINT-200U19, ts_keyboards:MX-FPRINT-1900-200U
- removed Z15, Z28: MX-FPRINT-150U19, ts_keyboards:MX-FPRINT-1900-150U
- removed Z29: MX-FPRINT-175U19, ts_keyboards:MX-FPRINT-1900-175U
- removed Z41, Z42: MX-FPRINT-225U19, ts_keyboards:MX-FPRINT-1900-225U
- removed Z53: MX-FPRINT-275U19, ts_keyboards:MX-FPRINT-1900-275U
- removed Z54, Z55, Z56, Z58, Z59, Z60, Z61: MX-FPRINT-125U19, ts_keyboards:MX-FPRINT-1900-125U
- removed Z57: MX-FPRINT-625U19, ts_keyboards:MX-FPRINT-1900-625U
- added IC1: MC74VHC1G50SC-74A, ts_keyboards:SC-74A
- added S_APP, S_BSLS, S_BSPC, S_CAPS, S_LALT, S_LBRC, S_LCTL, S_LGUI, S_LSFT, S_MINS, S_QUOT, S_RALT, S_RBRC, S_RCTL, S_RSFT, S_SCLN, S_SLSH: MX-5-PIN-HOTSWAP-PAD, ts_keyboards:MX-5-PIN-HOTSWAP-PAD
- added T_BSPC, T_ENT, T_LSFT, T_RSFT: MX-STABS-200U, ts_keyboards:MX-STABS-200U
- added T_SPC: MX-STABS-625U, ts_keyboards:MX-STABS-625U
- moved S_ENT 0.70 mm to (264.3, 47.6)
- moved S_EQL 0.66 mm to (238.1, 85.7)
- moved X1 0.60 mm to (78.7, 61.6)
- moved S_P 0.58 mm to (209.6, 66.7)
- moved S_0 0.57 mm to (200.0, 85.7)
- moved S_DOT 0.54 mm to (204.8, 28.6)
- moved S_FN1 0.53 mm to (202.4, 9.53)
- moved S_O 0.53 mm to (190.5, 66.7)
- moved S_L 0.53 mm to (195.3, 47.6)
- moved S_9 0.53 mm to (181.0, 85.7)
- moved S_COM 0.49 mm to (185.7, 28.6)
- moved S_I 0.48 mm to (171.4, 66.7)
- moved S_8 0.48 mm to (161.9, 85.7)
- moved S_K 0.48 mm to (176.2, 47.6)
- moved S_M 0.44 mm to (166.7, 28.6)
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Connections:
- net GND: now also IC1.3; no longer Y1.1, Y1.3
- net LED1ST: now also IC1.2; no longer Y1.2
- net MY2: now also S_CAPS.P$2, S_CAPS.P$4; no longer S_CPS.P$2, S_CPS.P$4
- net MY3: now also S_LSFT.P$2, S_LSFT.P$4; no longer S_LSH.P$2, S_LSH.P$4
- net MY4: now also S_APP.P$2, S_APP.P$4, S_LALT.P$2, S_LALT.P$4, S_LCTL.P$2, S_LCTL.P$4, S_LGUI.P$2, S_LGUI.P$4, S_RALT.P$2, S_RALT.P$4, S_RCTL.P$2, S_RCTL.P$4; no longer S_LAL.P$2, S_LAL.P$4, S_LCT.P$2, S_LCT.P$4, S_LGU.P$2, S_LGU.P$4, S_RAL.P$2, S_RAL.P$4, S_RCT.P$2, S_RCT.P$4, S_RGU.P$2, S_RGU.P$4
- net MY5: now also S_BSPC.P$2, S_BSPC.P$4, S_MINS.P$2, S_MINS.P$4; no longer S_BSP.P$2, S_BSP.P$4, S_MIN.P$2, S_MIN.P$4
- net MY6: now also S_BSLS.P$2, S_BSLS.P$4, S_LBRC.P$2, S_LBRC.P$4, S_RBRC.P$2, S_RBRC.P$4; no longer S_BSL.P$2, S_BSL.P$4, S_CB.P$2, S_CB.P$4, S_OB.P$2, S_OB.P$4
- net MY7: now also S_QUOT.P$2, S_QUOT.P$4, S_SCLN.P$2, S_SCLN.P$4; no longer S_QUO.P$2, S_QUO.P$4, S_SCL.P$2, S_SCL.P$4
- net MY8: now also S_RSFT.P$2, S_RSFT.P$4, S_SLSH.P$2, S_SLSH.P$4; no longer S_FSL.P$2, S_FSL.P$4, S_RSH.P$2, S_RSH.P$4
- net N$12: now also S_MINS.P$1, S_MINS.P$3; no longer S_MIN.P$1, S_MIN.P$3
- net N$14: now also S_BSPC.P$1, S_BSPC.P$3; no longer S_BSP.P$1, S_BSP.P$3
- net N$26: now also S_LBRC.P$1, S_LBRC.P$3; no longer S_OB.P$1, S_OB.P$3
- net N$27: now also S_RBRC.P$1, S_RBRC.P$3; no longer S_CB.P$1, S_CB.P$3
- net N$28: now also S_BSLS.P$1, S_BSLS.P$3; no longer S_BSL.P$1, S_BSL.P$3
- net N$39: now also S_SCLN.P$1, S_SCLN.P$3; no longer S_SCL.P$1, S_SCL.P$3
- net N$40: now also S_QUOT.P$1, S_QUOT.P$3; no longer S_QUO.P$1, S_QUO.P$3
- net N$42: now also S_LSFT.P$1, S_LSFT.P$3; no longer S_LSH.P$1, S_LSH.P$3
- net N$52: now also S_SLSH.P$1, S_SLSH.P$3; no longer S_FSL.P$1, S_FSL.P$3
- net N$53: now also S_RSFT.P$1, S_RSFT.P$3; no longer S_RSH.P$1, S_RSH.P$3
- net N$54: now also S_LCTL.P$1, S_LCTL.P$3; no longer S_LCT.P$1, S_LCT.P$3
- net N$55: now also S_LGUI.P$1, S_LGUI.P$3; no longer S_LGU.P$1, S_LGU.P$3
- net N$56: now also S_LALT.P$1, S_LALT.P$3; no longer S_LAL.P$1, S_LAL.P$3
- net N$59: now also S_APP.P$1, S_APP.P$3; no longer S_RAL.P$1, S_RAL.P$3
- net N$60: now also S_RALT.P$1, S_RALT.P$3; no longer S_RGU.P$1, S_RGU.P$3
- net N$61: now also S_RCTL.P$1, S_RCTL.P$3; no longer S_RCT.P$1, S_RCT.P$3
- net N$62: now also S_CAPS.P$1, S_CAPS.P$3; no longer S_CPS.P$1, S_CPS.P$3
- net N$66: now also IC1.4; no longer Y1.4
- net VSUP: now also IC1.5; no longer Y1.5
Routing:
- net MX1: track 437.8 -> 0.00 mm, vias 13 -> 0
- net MX6: track 387.4 -> 0.00 mm, vias 6 -> 0
- net MX2: track 381.3 -> 0.00 mm, vias 7 -> 0
- net MY4: track 350.9 -> 0.00 mm, vias 1 -> 0
- net MX3: track 326.3 -> 0.00 mm, vias 7 -> 0
- net MX4: track 320.7 -> 0.00 mm, vias 5 -> 0
- net MX5: track 314.5 -> 0.00 mm, vias 9 -> 0
- net MX0: track 298.4 -> 0.00 mm, vias 8 -> 0
- net MX7: track 292.4 -> 0.00 mm, vias 8 -> 0
- net VSUP: track 256.5 -> 0.00 mm, vias 7 -> 0
- net MY2: track 247.6 -> 0.00 mm, vias 3 -> 0
- net MY6: track 231.3 -> 0.00 mm, vias 8 -> 0
- net !BOOT: track 216.1 -> 0.00 mm, vias 4 -> 0
- net MY8: track 209.9 -> 0.00 mm, vias 3 -> 0
- net MY7: track 205.1 -> 0.00 mm, vias 3 -> 0
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Other:
- board size 283 x 93 mm -> 283.8 x 93.3 mm

Commit message: wip 2022-07-22
Parts:
- removed SA1, SA2, SA3, SC2: MOUNTING-HOLE-WIDE, ts_keyboards:MOUNTING-HOLE-WIDE
- removed SC1: MOUNTING-HOLE, ts_keyboards:MOUNTING-HOLE
- removed SG1, SG4: MOUNTING-HOLE-VWIDEEDGE-CUT, ts_keyboards:MOUNTING-HOLE-VWIDE-C
- added FP_AP2: FOOTPRINT-AP2, ts_keyboards:FOOTPRINT-AP2
- added FP_GH60: FOOTPRINT-GH60, ts_keyboards:FOOTPRINT-GH60
- moved IC1 60.2 mm to (-2.50, 59.0), flipped to the bottom
- moved J2 44.2 mm to (-5.00, 75.0)
- moved JP1 35.2 mm to (-4.00, 66.0)
- moved PTC 24.0 mm to (-3.40, 87.5)
- moved ESD 23.4 mm to (-3.50, 92.9)
- moved TVS 20.6 mm to (-3.40, 82.8)
- moved D9 20.2 mm to (170.2, 76.7)
- moved D60 19.6 mm to (244.2, 4.67)
- moved D8 19.2 mm to (151.2, 76.7)
- moved D54 19.2 mm to (5.17, 4.67)
- moved JP2 17.5 mm to (-2.00, 63.0)
- moved D29 16.1 mm to (10.2, 42.7)
- moved D28 15.2 mm to (265.2, 61.7)
- moved D19 14.5 mm to (89.2, 61.7)
- moved C7 14.0 mm to (-3.00, 41.5)
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Connections:
- removed net SA1: SA1.P$10, SA1.P$2, SA1.P$3, SA1.P$4, SA1.P$5, SA1.P$7, SA1.P$8, SA1.P$9
- removed net SA2: SA2.P$10, SA2.P$2, SA2.P$3, SA2.P$4, SA2.P$5, SA2.P$7, SA2.P$8, SA2.P$9
- removed net SA3: SA3.P$10, SA3.P$2, SA3.P$3, SA3.P$4, SA3.P$5, SA3.P$7, SA3.P$8, SA3.P$9
- removed net SC2: SC2.P$10, SC2.P$2, SC2.P$3, SC2.P$4, SC2.P$5, SC2.P$7, SC2.P$8, SC2.P$9
- removed net SG1: SG1.P$1, SG1.P$4, SG1.P$5, SG1.P$6, SG1.P$7, SG1.P$8
- removed net SG4: SG4.P$1, SG4.P$4, SG4.P$5, SG4.P$6, SG4.P$7, SG4.P$8
- net SC1: no longer SC1.P$10, SC1.P$2, SC1.P$3, SC1.P$7, SC1.P$8, SC1.P$9
Other:
- board text added: "Rev B | Ver 2022-08-01"
- board text removed: "Rev B"
- board text removed: "Ver 1.0 | Rev 2022-06-06"

Commit message: final touches and validation for rev B
Parts:
- removed IC1: MC74VHC1G50SC-74A, ts_keyboards:SC-74A
- added D62: (no value), jlcpcb_basic_parts:SOD-123
- added J6: (no value), SparkFun-Connectors:1X01
- added J7: (no value), SparkFun-Connectors:1X02
- added S_BSLS2, S_ENT2, S_LSFT2, S_NUBS: MX-5-PIN-HOTSWAP-PADNO-SILK, ts_keyboards:MX-5-PIN-HOTSWAP-PAD-NS
- added T_ENT1: MX-STABS-200U, ts_keyboards:MX-STABS-200U
- added U$14: 74AHCT1G125GV, ts_keyboards:SC-74A
- J3: device SparkFun-Connectors:1X04 -> SparkFun-Connectors:1X03
- moved D54 248.7 mm to (253.2, 23.7)
- moved C7 177.3 mm to (168.0, 88.5), turned to 180 degrees
- moved C11 156.5 mm to (21.0, 38.5)
- moved JP1 75.3 mm to (55.6, 19.9), turned to 0 degrees
- moved D58 72.0 mm to (124.2, 4.67)
- moved D57 71.0 mm to (53.2, 4.67)
- moved J3 70.0 mm to (123.5, 64.0), flipped to the bottom, turned to 270 degrees
- moved J2 48.2 mm to (43.0, 79.0)
- moved R3 45.3 mm to (59.4, 19.9), turned to 0 degrees
- moved R4 45.1 mm to (63.6, 19.9), turned to 0 degrees
- moved C12 43.2 mm to (39.8, 40.0), turned to 180 degrees
- moved C10 39.0 mm to (111.0, 88.5)
- moved D0 38.5 mm to (39.2, 61.5)
- moved C8 37.0 mm to (149.0, 88.5)
- moved D53 36.0 mm to (217.2, 23.7)
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Connections:
- removed net A0: J3.3, X1.34
- removed net PWM: J3.2, X1.32
- removed net SINK: LM1117.4
- removed net SWDCK: X1.21
- removed net SWDIO: X1.23
- new net 52: J3.2, X1.52
- new net 63: J6.1, X1.63
- new net N$69: D43.A, S_NUBS.P$1, S_NUBS.P$3
- new net USBHOST_D+: J7.1, X1.35
- new net USBHOST_D-: J7.2, X1.37
- net GND: now also U$14.1, U$14.3; no longer IC1.3
- net LED: now also X1.32; no longer X1.47
- net LED1ST: now also U$14.2; no longer IC1.2
- net MX0: now also D50.C, D55.C, X1.47; no longer D49.C, D54.C, X1.18
- net MX1: now also D43.C, D51.C, D56.C, X1.19; no longer D50.C, D55.C, X1.16
- net MX2: now also D44.C, D52.C, D57.C, X1.17; no longer D43.C, D51.C, D56.C, X1.14
- net MX3: now also D45.C, D53.C, D58.C, X1.18; no longer D44.C, D52.C, D57.C, X1.38
- net MX4: now also D46.C, D59.C, X1.16; no longer D45.C, D58.C, X1.12
- net MX5: now also D47.C, D54.C, D60.C, X1.14; no longer D46.C, D53.C, D59.C, X1.10
- net MX6: now also D48.C, D61.C, X1.12; no longer D47.C, D60.C, X1.17
- net MX7: now also D49.C, D62.C, X1.10; no longer D48.C, D61.C, X1.19
- net MY2: now also X1.50; no longer X1.52
- net MY3: now also S_LSFT2.P$2, S_LSFT2.P$4, S_NUBS.P$2, S_NUBS.P$4, X1.46; no longer X1.50
- net MY4: now also X1.44; no longer X1.48
- net MY5: now also X1.42; no longer X1.46
- net MY6: now also S_BSLS2.P$2, S_BSLS2.P$4, X1.40; no longer X1.44
- net MY7: now also S_ENT2.P$2, S_ENT2.P$4, X1.38; no longer X1.42
- net MY8: now also X1.34; no longer X1.40
- net N$28: now also S_BSLS2.P$1, S_BSLS2.P$3
- net N$41: now also S_ENT2.P$1, S_ENT2.P$3
- net N$42: now also S_LSFT2.P$1, S_LSFT2.P$3
- net N$43: now also D44.A; no longer D43.A
- net N$44: now also D45.A; no longer D44.A
- net N$45: now also D46.A; no longer D45.A
- net N$46: now also D47.A; no longer D46.A
- net N$47: now also D48.A; no longer D47.A
- net N$48: now also D49.A; no longer D48.A
- net N$49: now also D50.A; no longer D49.A
- net N$50: now also D51.A; no longer D50.A
- net N$51: now also D52.A; no longer D51.A
- net N$52: now also D53.A; no longer D52.A
- net N$53: now also D54.A; no longer D53.A
- net N$54: now also D55.A; no longer D54.A
- net N$55: now also D56.A; no longer D55.A
- net N$56: now also D57.A; no longer D56.A
- net N$57: now also D58.A; no longer D57.A
- net N$58: now also D59.A; no longer D58.A
- net N$59: now also D60.A; no longer D59.A
- net N$60: now also D61.A; no longer D60.A
- net N$61: now also D62.A; no longer D61.A
- net N$66: now also U$14.4; no longer IC1.4
- net VCC: now also J3.3; no longer J3.4
- net VSUP: now also U$14.6; no longer IC1.5
Routing:
- net MX6: track 0.00 -> 463.9 mm, vias 0 -> 20
- net MX3: track 0.00 -> 431.0 mm, vias 0 -> 10
- net MX0: track 0.00 -> 405.8 mm, vias 0 -> 12
- net VSUP: track 0.00 -> 405.7 mm, vias 0 -> 19
- net MX1: track 0.00 -> 401.8 mm, vias 0 -> 11
- net MX2: track 0.00 -> 393.0 mm, vias 0 -> 13
- net MX4: track 0.00 -> 376.0 mm, vias 0 -> 14
- net MX7: track 0.00 -> 368.0 mm, vias 0 -> 11
- net MX5: track 0.00 -> 366.2 mm, vias 0 -> 14
- net MY5: track 0.00 -> 342.7 mm, vias 0 -> 15
- net MY4: track 0.00 -> 342.5 mm, vias 0 -> 4
- net MY6: track 0.00 -> 287.5 mm, vias 0 -> 6
- net MY7: track 0.00 -> 266.3 mm, vias 0 -> 4
- net MY3: track 0.00 -> 253.9 mm, vias 0 -> 6
- net MY0: track 0.00 -> 251.7 mm, vias 0 -> 9
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Other:
- board text added: "52"
- board text added: "63"
- board text added: "EEPROM"
- board text added: "HD+"
- board text added: "HD-"
- board text added: "JLCJLCJLCJLC"
- board text added: "Rev B | Ver 2022-08-27"
- board text removed: "A0"
- board text removed: "PWM"
- board text removed: "Rev B | Ver 2022-08-01"
- board text removed: "V/REG"

Commit message: updates after production prep
Parts:
- C12: value 1mF -> 0.1uF
- renumbered C1 to C01, C2 to C02, C3 to C03, C4 to C04, C5 to C05, C6 to C06, C7 to C07, C8 to C08, C9 to C09, D0 to D00, D1 to D01, D2 to D02, D3 to D03, D4 to D04, D5 to D05, D6 to D06, D7 to D07, D8 to D08, D9 to D09, J1 to J-BOOT, J2 to J-UDB, J3 to J-52, J4 to J-LED, J5 to J-UBS, J6 to J-63, J7 to J-HOST, JP1 to JP-VIN3, JP2 to JP-GND, W1 to M1

Commit message: move r8 + final rev B production files
Parts:
- moved R8 2.00 mm to (92.4, 54.7)
Routing:
- net SCK: track 19.1 -> 20.8 mm
Other:
- board text added: "ESD"
- board text added: "PTC"
Changed lines of the file:
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@@
 <text x="138.4" y="60.5" size="1.778" layer="22" rot="MR0" align="bottom-center">AP2</text>
 <text x="260.4" y="63.1" size="1.778" layer="22" rot="MR0" align="top-center">CMN</text>
-<text x="22.3" y="63.5" size="1.778" layer="22" rot="MR135" align="center-right">GROUND</text>
+<text x="23.2" y="62.9" size="1.778" layer="22" rot="MR180" align="center-right">GROUND</text>
 <text x="163.9" y="8.6" size="1.778" layer="22" rot="MR0">BOOT</text>
-<text x="29.4" y="50" size="1.778" layer="22" rot="MR90" align="center-left">BOOT</text>
-<text x="29.5" y="37.5" size="1.778" layer="22" rot="MR90" align="center-right">RESET</text>
+<text x="29.7" y="50" size="1.778" layer="22" rot="MR90" align="center-left">BOOT</text>
+<text x="29.8" y="37.5" size="1.778" layer="22" rot="MR90" align="center-right">RESET</text>
 <hole x="189.5" y="9.6" drill="2.5"/>
 <hole x="191.5" y="9.6" drill="2.5"/>
@@
 <circle x="9.45" y="35.55" radius="2" width="0.5" layer="22"/>
 <text x="283.2" y="92.7" size="1.778" layer="22" rot="MR270">JLCJLCJLCJLC</text>
+<circle x="20.6" y="75.8" radius="0.2" width="0.1524" layer="22"/>
+<circle x="41" y="37.6" radius="0.2" width="0.1524" layer="22"/>
+<text x="27.1" y="76.9" size="1" layer="26" rot="MR0">PTC</text>
+<text x="16.6" y="78.4" size="1" layer="26" rot="MR270">ESD</text>
 </plain>
 <attributes>
@@
 </element>
 <element name="JP-VIN3" library="SparkFun-Jumpers" library_urn="urn:adsk.eagle:library:528" package="SMT-JUMPER_2_NC_PASTE_NO-SILK" package3d_urn="urn:adsk.eagle:package:39283/1" value="OPT" x="55.6" y="19.9" smashed="yes" rot="MR0">
-<attribute name="NAME" x="55.6" y="21.543" size="1" layer="26" font="vector" ratio="20" rot="MR0" align="bottom-center"/>
+<attribute name="NAME" x="53.6" y="21.543" size="1" layer="26" font="vector" ratio="20" rot="MR0" align="bottom-center"/>
 <attribute name="VALUE" x="55.6" y="18.757" size="0.6096" layer="28" font="vector" ratio="20" rot="MR0" align="top-center"/>
 </element>
@@
 <attribute name="VALUE" x="95.3" y="59.86" size="0.6096" layer="28" font="vector" ratio="20" rot="MR180" align="bottom-center"/>
 </element>
-<element name="R8" library="rcl" library_urn="urn:adsk.eagle:library:334" package="R0603" package3d_urn="urn:adsk.eagle:package:23555/3" value="5.1K" x="94.4" y="54.7" smashed="yes" rot="MR180">
+<element name="R8" library="rcl" library_urn="urn:adsk.eagle:library:334" package="R0603" package3d_urn="urn:adsk.eagle:package:23555/3" value="5.1K" x="92.4" y="54.7" smashed="yes" rot="MR180">
 <attribute name="NAME" x="93.765" y="54.065" size="1.27" layer="26" rot="MR180"/>
 <attribute name="POPULARITY" value="70" x="94.4" y="54.7" size="1.778" layer="28" rot="MR180" display="off"/>
@@
 <element name="T_ENT1" library="ts_keyboards" package="MX-STABS-200U" value="MX-STABS-200U" x="273.844" y="57.15" smashed="yes" rot="R270"/>
 <element name="J-52" library="SparkFun-Connectors" library_urn="urn:adsk.eagle:library:513" package="1X03" package3d_urn="urn:adsk.eagle:package:38063/1" value="" x="123.5" y="64" smashed="yes" rot="MR270">
-<attribute name="NAME" x="122.103" y="65.27" size="0.6096" layer="26" font="vector" ratio="20" rot="MR270"/>
 <attribute name="VALUE" x="125.532" y="65.27" size="0.6096" layer="28" font="vector" ratio="20" rot="MR270"/>
 </element>
@@
 <wire x1="95.95" y1="57.215" x2="95.935" y2="57.2" width="0.254" layer="16"/>
 <wire x1="84.025" y1="59" x2="95.35" y2="59" width="0.254" layer="16"/>
-<wire x1="95.935" y1="57.2" x2="95.935" y2="55.385" width="0.254" layer="16"/>
-<wire x1="95.935" y1="55.385" x2="95.25" y2="54.7" width="0.254" layer="16"/>
+<wire x1="95.935" y1="57.2" x2="96" y2="57.135" width="0.254" layer="16"/>
+<wire x1="96" y1="57.135" x2="96" y2="56" width="0.254" layer="16"/>
+<wire x1="94.7" y1="54.7" x2="93.25" y2="54.7" width="0.254" layer="16"/>
+<wire x1="96" y1="56" x2="94.7" y2="54.7" width="0.254" layer="16"/>
 </signal>
 <signal name="EE_CS">
