File: EAGLE/vr61/vr61-revB.brd (EAGLE design)
At the start: 283.8 x 93.3 mm, 191 parts, among them M1 M25C, X1 MICROMOD-2222-C

Commit message: minor edits
Parts:
- added S3: BOOT, SparkFun-Switches:TACTILE_SWITCH_SMD_5.2MM
Connections:
- net !BOOT: now also S3.3, S3.4
- net GND: now also S3.1, S3.2
Routing:
- net !BOOT: track 202.9 -> 207.7 mm
- net MX6: track 463.9 -> 466.2 mm
- net MX5: track 366.2 -> 367.6 mm

Commit message: Reb B.2 update
Parts:
- removed JP-VIN3: OPT, SparkFun-Jumpers:SMT-JUMPER_2_NC_PASTE_NO-SILK
- added D63, D64, D65, D66, D67: (no value), jlcpcb_basic_parts:SOD-123
- added DIP-SW: DIP004, untitled:DIP-1.27-004
- added J-VIN: (no value), ts_jumpers:SOLDERJUMPER_ARROW_NOPASTE
- added S_BSPC2, S_CAPS2, S_FN, S_RSFT2, S_SPARE: MX-5-PIN-MILMAX-3305-XNO-SILK, ts_keyboards:MX-5-PIN-MILMAX-3305-X-NS
- added U$20, U$21, U$22: FIDUCIAL, __temp_to_delete:FIDUCIAL
- JP-GND: device SparkFun-Jumpers:SMT-JUMPER_2_NO_NO-SILK -> ts_jumpers:SOLDERJUMPER_ARROW_NOPASTE
- moved R3 54.5 mm to (107.8, 44.8), turned to 180 degrees
- moved R4 49.7 mm to (107.8, 42.7)
- moved U$8 10.0 mm to (139.0, 6.00)
- moved D20 9.06 mm to (117.2, 62.7)
- moved D29 3.00 mm to (10.2, 39.7)
- moved D28 2.83 mm to (264.2, 78.5)
- moved JP-GND 0.83 mm to (25.4, 59.5), turned to 270 degrees
- turned C11 to 0 degrees
Connections:
- removed net N$68: JP-VIN3.1, R3.2
- new net N$70: D64.A, S_SPARE.1
- new net N$71: D63.A, S_FN.1
- new net N$73: D65.A, DIP-SW.1
- new net N$74: DIP-SW.4, J-VIN.2, R3.2
- new net N$75: D66.A, DIP-SW.2
- new net N$76: D67.A, DIP-SW.3
- net GROUND: now also JP-GND.2; no longer JP-GND.1
- net MX4: now also D63.C, D64.C
- net MX5: now also D65.C, D66.C, D67.C
- net MY0: now also S_1.2@1, S_1.2@2, S_2.2@1, S_2.2@2, S_3.2@1, S_3.2@2, S_4.2@1, S_4.2@2, S_5.2@1, S_5.2@2, S_6.2@1, S_6.2@2, S_7.2@1, S_7.2@2, S_ESC.2@1, S_ESC.2@2; no longer S_1.P$2, S_1.P$4, S_2.P$2, S_2.P$4, S_3.P$2, S_3.P$4, S_4.P$2, S_4.P$4, S_5.P$2, S_5.P$4, S_6.P$2, S_6.P$4, S_7.P$2, S_7.P$4, S_ESC.P$2, S_ESC.P$4
- net MY1: now also S_E.2@1, S_E.2@2, S_Q.2@1, S_Q.2@2, S_R.2@1, S_R.2@2, S_T.2@1, S_T.2@2, S_TAB.2@1, S_TAB.2@2, S_U.2@1, S_U.2@2, S_W.2@1, S_W.2@2, S_Y.2@1, S_Y.2@2; no longer S_E.P$2, S_E.P$4, S_Q.P$2, S_Q.P$4, S_R.P$2, S_R.P$4, S_T.P$2, S_T.P$4, S_TAB.P$2, S_TAB.P$4, S_U.P$2, S_U.P$4, S_W.P$2, S_W.P$4, S_Y.P$2, S_Y.P$4
- net MY2: now also S_A.2@1, S_A.2@2, S_CAPS.2@1, S_CAPS.2@2, S_CAPS2.1, S_D.2@1, S_D.2@2, S_F.2@1, S_F.2@2, S_G.2@1, S_G.2@2, S_H.2@1, S_H.2@2, S_J.2@1, S_J.2@2, S_S.2@1, S_S.2@2; no longer S_A.P$2, S_A.P$4, S_CAPS.P$2, S_CAPS.P$4, S_D.P$2, S_D.P$4, S_F.P$2, S_F.P$4, S_G.P$2, S_G.P$4, S_H.P$2, S_H.P$4, S_J.P$2, S_J.P$4, S_S.P$2, S_S.P$4
- net MY3: now also S_B.2@1, S_B.2@2, S_C.2@1, S_C.2@2, S_LSFT.2@1, S_LSFT.2@2, S_LSFT2.2@1, S_LSFT2.2@2, S_N.2@1, S_N.2@2, S_NUBS.2@1, S_NUBS.2@2, S_V.2@1, S_V.2@2, S_X.2@1, S_X.2@2, S_Z.2@1, S_Z.2@2; no longer S_B.P$2, S_B.P$4, S_C.P$2, S_C.P$4, S_LSFT.P$2, S_LSFT.P$4, S_LSFT2.P$2, S_LSFT2.P$4, S_N.P$2, S_N.P$4, S_NUBS.P$2, S_NUBS.P$4, S_V.P$2, S_V.P$4, S_X.P$2, S_X.P$4, S_Z.P$2, S_Z.P$4
- net MY4: now also S_APP.2@1, S_APP.2@2, S_FN1.2@1, S_FN1.2@2, S_LALT.2@1, S_LALT.2@2, S_LCTL.2@1, S_LCTL.2@2, S_LGUI.2@1, S_LGUI.2@2, S_RALT.2@1, S_RALT.2@2, S_RCTL.2@1, S_RCTL.2@2, S_SPC.2@1, S_SPC.2@2; no longer S_APP.P$2, S_APP.P$4, S_FN1.P$2, S_FN1.P$4, S_LALT.P$2, S_LALT.P$4, S_LCTL.P$2, S_LCTL.P$4, S_LGUI.P$2, S_LGUI.P$4, S_RALT.P$2, S_RALT.P$4, S_RCTL.P$2, S_RCTL.P$4, S_SPC.P$2, S_SPC.P$4
- net MY5: now also DIP-SW.8, S_0.2@1, S_0.2@2, S_8.2@1, S_8.2@2, S_9.2@1, S_9.2@2, S_BSPC.2@1, S_BSPC.2@2, S_BSPC2.2, S_EQL.2@1, S_EQL.2@2, S_MINS.2@1, S_MINS.2@2; no longer S_0.P$2, S_0.P$4, S_8.P$2, S_8.P$4, S_9.P$2, S_9.P$4, S_BSPC.P$2, S_BSPC.P$4, S_EQL.P$2, S_EQL.P$4, S_MINS.P$2, S_MINS.P$4
- net MY6: now also DIP-SW.7, S_BSLS.2@1, S_BSLS.2@2, S_BSLS2.2@1, S_BSLS2.2@2, S_I.2@1, S_I.2@2, S_LBRC.2@1, S_LBRC.2@2, S_O.2@1, S_O.2@2, S_P.2@1, S_P.2@2, S_RBRC.2@1, S_RBRC.2@2; no longer S_BSLS.P$2, S_BSLS.P$4, S_BSLS2.P$2, S_BSLS2.P$4, S_I.P$2, S_I.P$4, S_LBRC.P$2, S_LBRC.P$4, S_O.P$2, S_O.P$4, S_P.P$2, S_P.P$4, S_RBRC.P$2, S_RBRC.P$4
- net MY7: now also DIP-SW.6, S_ENT.2@1, S_ENT.2@2, S_ENT2.2@1, S_ENT2.2@2, S_K.2@1, S_K.2@2, S_L.2@1, S_L.2@2, S_QUOT.2@1, S_QUOT.2@2, S_SCLN.2@1, S_SCLN.2@2, S_SPARE.2; no longer S_ENT.P$2, S_ENT.P$4, S_ENT2.P$2, S_ENT2.P$4, S_K.P$2, S_K.P$4, S_L.P$2, S_L.P$4, S_QUOT.P$2, S_QUOT.P$4, S_SCLN.P$2, S_SCLN.P$4
- net MY8: now also S_COM.2@1, S_COM.2@2, S_DOT.2@1, S_DOT.2@2, S_FN.2, S_M.2@1, S_M.2@2, S_RSFT.2@1, S_RSFT.2@2, S_RSFT2.2, S_SLSH.2@1, S_SLSH.2@2; no longer S_COM.P$2, S_COM.P$4, S_DOT.P$2, S_DOT.P$4, S_M.P$2, S_M.P$4, S_RSFT.P$2, S_RSFT.P$4, S_SLSH.P$2, S_SLSH.P$4
- net N$1: now also S_ESC.1@1, S_ESC.1@2; no longer S_ESC.P$1, S_ESC.P$3
- net N$10: now also S_9.1@1, S_9.1@2; no longer S_9.P$1, S_9.P$3
- net N$11: now also S_0.1@1, S_0.1@2; no longer S_0.P$1, S_0.P$3
- net N$12: now also S_MINS.1@1, S_MINS.1@2; no longer S_MINS.P$1, S_MINS.P$3
- net N$13: now also S_EQL.1@1, S_EQL.1@2; no longer S_EQL.P$1, S_EQL.P$3
- net N$14: now also S_BSPC.1@1, S_BSPC.1@2, S_BSPC2.1; no longer S_BSPC.P$1, S_BSPC.P$3
- net N$15: now also S_TAB.1@1, S_TAB.1@2; no longer S_TAB.P$1, S_TAB.P$3
- net N$16: now also S_Q.1@1, S_Q.1@2; no longer S_Q.P$1, S_Q.P$3
- net N$17: now also S_W.1@1, S_W.1@2; no longer S_W.P$1, S_W.P$3
- net N$18: now also S_E.1@1, S_E.1@2; no longer S_E.P$1, S_E.P$3
- net N$19: now also S_R.1@1, S_R.1@2; no longer S_R.P$1, S_R.P$3
- net N$2: now also S_1.1@1, S_1.1@2; no longer S_1.P$1, S_1.P$3
- net N$20: now also S_T.1@1, S_T.1@2; no longer S_T.P$1, S_T.P$3
- net N$21: now also S_Y.1@1, S_Y.1@2; no longer S_Y.P$1, S_Y.P$3
- net N$22: now also S_U.1@1, S_U.1@2; no longer S_U.P$1, S_U.P$3
- net N$23: now also S_I.1@1, S_I.1@2; no longer S_I.P$1, S_I.P$3
- net N$24: now also S_O.1@1, S_O.1@2; no longer S_O.P$1, S_O.P$3
- net N$25: now also S_P.1@1, S_P.1@2; no longer S_P.P$1, S_P.P$3
- net N$26: now also S_LBRC.1@1, S_LBRC.1@2; no longer S_LBRC.P$1, S_LBRC.P$3
- net N$27: now also S_RBRC.1@1, S_RBRC.1@2; no longer S_RBRC.P$1, S_RBRC.P$3
- net N$28: now also S_BSLS.1@1, S_BSLS.1@2, S_BSLS2.1@1, S_BSLS2.1@2; no longer S_BSLS.P$1, S_BSLS.P$3, S_BSLS2.P$1, S_BSLS2.P$3
- net N$3: now also S_2.1@1, S_2.1@2; no longer S_2.P$1, S_2.P$3
- net N$30: now also S_A.1@1, S_A.1@2; no longer S_A.P$1, S_A.P$3
- net N$31: now also S_S.1@1, S_S.1@2; no longer S_S.P$1, S_S.P$3
- net N$32: now also S_D.1@1, S_D.1@2; no longer S_D.P$1, S_D.P$3
- net N$33: now also S_F.1@1, S_F.1@2; no longer S_F.P$1, S_F.P$3
- net N$34: now also S_G.1@1, S_G.1@2; no longer S_G.P$1, S_G.P$3
- net N$35: now also S_H.1@1, S_H.1@2; no longer S_H.P$1, S_H.P$3
- net N$36: now also S_J.1@1, S_J.1@2; no longer S_J.P$1, S_J.P$3
- net N$37: now also S_K.1@1, S_K.1@2; no longer S_K.P$1, S_K.P$3
- net N$38: now also S_L.1@1, S_L.1@2; no longer S_L.P$1, S_L.P$3
- net N$39: now also S_SCLN.1@1, S_SCLN.1@2; no longer S_SCLN.P$1, S_SCLN.P$3
- net N$4: now also S_3.1@1, S_3.1@2; no longer S_3.P$1, S_3.P$3
- net N$40: now also S_QUOT.1@1, S_QUOT.1@2; no longer S_QUOT.P$1, S_QUOT.P$3
- net N$41: now also S_ENT.1@1, S_ENT.1@2, S_ENT2.1@1, S_ENT2.1@2; no longer S_ENT.P$1, S_ENT.P$3, S_ENT2.P$1, S_ENT2.P$3
- net N$42: now also S_LSFT.1@1, S_LSFT.1@2, S_LSFT2.1@1, S_LSFT2.1@2; no longer S_LSFT.P$1, S_LSFT.P$3, S_LSFT2.P$1, S_LSFT2.P$3
- net N$43: now also S_Z.1@1, S_Z.1@2; no longer S_Z.P$1, S_Z.P$3
- net N$44: now also S_X.1@1, S_X.1@2; no longer S_X.P$1, S_X.P$3
- net N$45: now also S_C.1@1, S_C.1@2; no longer S_C.P$1, S_C.P$3
- net N$46: now also S_V.1@1, S_V.1@2; no longer S_V.P$1, S_V.P$3
- net N$47: now also S_B.1@1, S_B.1@2; no longer S_B.P$1, S_B.P$3
- net N$48: now also S_N.1@1, S_N.1@2; no longer S_N.P$1, S_N.P$3
- net N$49: now also S_M.1@1, S_M.1@2; no longer S_M.P$1, S_M.P$3
- net N$5: now also S_4.1@1, S_4.1@2; no longer S_4.P$1, S_4.P$3
- net N$50: now also S_COM.1@1, S_COM.1@2; no longer S_COM.P$1, S_COM.P$3
- net N$51: now also S_DOT.1@1, S_DOT.1@2; no longer S_DOT.P$1, S_DOT.P$3
- net N$52: now also S_SLSH.1@1, S_SLSH.1@2; no longer S_SLSH.P$1, S_SLSH.P$3
- net N$53: now also S_RSFT.1@1, S_RSFT.1@2, S_RSFT2.1; no longer S_RSFT.P$1, S_RSFT.P$3
- net N$54: now also S_LCTL.1@1, S_LCTL.1@2; no longer S_LCTL.P$1, S_LCTL.P$3
- net N$55: now also S_LGUI.1@1, S_LGUI.1@2; no longer S_LGUI.P$1, S_LGUI.P$3
- net N$56: now also S_LALT.1@1, S_LALT.1@2; no longer S_LALT.P$1, S_LALT.P$3
- net N$57: now also S_SPC.1@1, S_SPC.1@2; no longer S_SPC.P$1, S_SPC.P$3
- net N$58: now also S_FN1.1@1, S_FN1.1@2; no longer S_FN1.P$1, S_FN1.P$3
- net N$59: now also S_APP.1@1, S_APP.1@2; no longer S_APP.P$1, S_APP.P$3
- net N$6: now also S_5.1@1, S_5.1@2; no longer S_5.P$1, S_5.P$3
- net N$60: now also S_RALT.1@1, S_RALT.1@2; no longer S_RALT.P$1, S_RALT.P$3
- net N$61: now also S_RCTL.1@1, S_RCTL.1@2; no longer S_RCTL.P$1, S_RCTL.P$3
- net N$62: now also S_CAPS.1@1, S_CAPS.1@2, S_CAPS2.2; no longer S_CAPS.P$1, S_CAPS.P$3
- net N$69: now also S_NUBS.1@1, S_NUBS.1@2; no longer S_NUBS.P$1, S_NUBS.P$3
- net N$7: now also S_6.1@1, S_6.1@2; no longer S_6.P$1, S_6.P$3
- net N$8: now also S_7.1@1, S_7.1@2; no longer S_7.P$1, S_7.P$3
- net N$9: now also S_8.1@1, S_8.1@2; no longer S_8.P$1, S_8.P$3
- net SC1: now also JP-GND.1; no longer JP-GND.2
- net VSUP: now also DIP-SW.5, J-VIN.1; no longer JP-VIN3.2
Routing:
- net MX4: track 376.0 -> 468.5 mm, vias 14 -> 18
- net MY7: track 266.3 -> 340.3 mm, vias 4 -> 7
- net MY8: track 251.3 -> 306.1 mm
- net MY5: track 342.7 -> 396.2 mm, vias 15 -> 16
- net GND: track 3.82 -> 52.2 mm, vias 28 -> 116
- net MY2: track 241.7 -> 290.0 mm, vias 6 -> 4
- net MY6: track 287.5 -> 330.3 mm, vias 6 -> 9
- net MY0: track 251.7 -> 292.6 mm
- net MY1: track 166.5 -> 194.5 mm
- net MY4: track 342.5 -> 368.9 mm
- net MY3: track 253.9 -> 280.2 mm
- net N$14: track 8.82 -> 32.4 mm
- net N$74: track 0.00 -> 21.8 mm, vias 0 -> 2
- net N$62: track 7.92 -> 28.5 mm
- net N$28: track 74.1 -> 89.6 mm
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Other:
- outline, holes or cut-outs redrawn
- board text added: "Rev B.2 | Ver 2024-09-17"
- board text added: "and"
- board text removed: "AP-3 x136.2 y57.9 d2.5"
- board text removed: "Rev B | Ver 2022-08-27"
- board text removed: "VIN/3"

Commit message: Boot switch redo
Parts:
- added C14: 100nF, rcl:C0603
- added D80: BAS70-05, diode:SOT23
- added R9: 5.1K, rcl:R0603
- added S4: BOOT, SparkFun-Switches:TACTILE_SWITCH_SMD_5.2MM
- S1: value Reset -> (none); device SparkFun-Switches:TACTILE_SWITCH_SMD_5.2MM -> VinoRodrigues_Custom_Eagle:SKRKAEE020
- S2: value BOOT -> (none); device SparkFun-Switches:TACTILE_SWITCH_SMD_5.2MM -> VinoRodrigues_Custom_Eagle:SKRKAEE020
- moved S3 142.2 mm to (29.5, 46.7), flipped to the bottom, turned to 0 degrees
- moved S2 34.6 mm to (61.5, 60.0), turned to 90 degrees
- moved S1 34.4 mm to (58.0, 60.0), turned to 90 degrees
- moved D17 13.7 mm to (56.7, 75.7)
Connections:
- new net BOOT: D80.3, J-BOOT.1, R9.1, S3.3, S3.4, S4.3, S4.4
- net !BOOT: now also C14.1, D80.1, S2.2; no longer J-BOOT.1, S2.3, S2.4, S3.3, S3.4
- net !RESET: now also D80.2, S1.2; no longer S1.3, S1.4
- net GND: now also C14.2, S4.1, S4.2; no longer S1.2, S2.2
- net VCC: now also R9.2
Routing:
- net BOOT: track 0.00 -> 186.5 mm, vias 0 -> 3
- net !BOOT: track 208.4 -> 74.7 mm, vias 7 -> 6
- net VCC: track 149.0 -> 178.3 mm, vias 10 -> 12
- net VSUP: track 397.8 -> 402.4 mm, vias 21 -> 25
- net N$17: track 14.8 -> 10.6 mm
- net MX2: track 392.8 -> 396.9 mm
- net MY1: track 194.5 -> 197.9 mm
- net !RESET: track 61.5 -> 62.8 mm, vias 6 -> 4
- net MY2: vias 4 -> 5
- net GND: vias 116 -> 119
Other:
- board text added: "!BOOT"
- board text added: "'"
- board text added: ","
- board text added: "-"
- board text added: "--6.25--"
- board text added: "--ANSI--"
- board text added: "--ISO--"
- board text added: "."
- board text added: "/"
- board text added: "0"
- board text added: "1"
- board text added: "2"
- board text added: "3"
- board text added: "4"
- board text added: "5"
- board text added: "6"
- board text added: "7"
- board text added: "8"
- board text added: "9"
- board text added: ";"
- board text added: "="
- board text added: "A"
- board text added: "ANSI"
- board text added: "Alt Cmd"
- board text added: "B"
- board text added: "Bspc"
- board text added: "C"
- board text added: "COMBO"
- board text added: "Caps"
- board text added: "Ctrl"
- board text added: "D"
- board text added: "E"
- board text added: "Ent"
- board text added: "Esc"
- board text added: "F"
- board text added: "Fn"
- board text added: "G"
- board text added: "H"
- board text added: "I"
- board text added: "ISO"
- board text added: "J"
- board text added: "K"
- board text added: "L"
- board text added: "M"
- board text added: "Menu Opt"
- board text added: "N"
- board text added: "NUBS"
- board text added: "NUHS"
- board text added: "O"
- board text added: "P"
- board text added: "Q"
- board text added: "R"
- board text added: "S"
- board text added: "Shft"
- board text added: "T"
- board text added: "Tab"
- board text added: "U"
- board text added: "V"
- board text added: "W"
- board text added: "Win Opt"
- board text added: "X"
- board text added: "Y"
- board text added: "Z"
- board text added: "["
- board text added: "\\"
- board text added: "]"

Commit message: .
Routing:
- net GND: track 52.2 -> 75.8 mm, vias 119 -> 120

Commit message: Added Bakeneko footprint
Parts:
- removed FP_GH60: FOOTPRINT-GH60, ts_keyboards:FOOTPRINT-GH60
- added U$24: FOOTPRINT-BAKENEKO60, ts_keyboards:FOOTPRINT-BAKENEKO60
- added U$25: FOOTPRINT-DIMS-GH60, ts_keyboards:FOOTPRINT-DIMS-GH60
- moved U$21 9.52 mm to (259.5, 92.0)
- moved D57 3.83 mm to (57.0, 4.64)
- moved D03 2.78 mm to (32.4, 91.7)
- moved D55 1.13 mm to (19.0, 5.80)
- moved D62 1.12 mm to (267.2, 5.80)
- moved R2 1.10 mm to (26.0, 90.3)
- moved R1 1.00 mm to (11.3, 90.3)
- moved R5 0.44 mm to (5.80, 90.9), turned to 180 degrees
- moved J-UBS 0.31 mm to (18.4, 88.3)
- moved S3 0.21 mm to (29.3, 46.6)
- turned C06 to 0 degrees
- renumbered U$14 to 74AH
Routing:
- net GND: track 75.8 -> 42.9 mm, vias 120 -> 127
- net GROUND: track 75.3 -> 71.4 mm
- net N$56: track 21.2 -> 25.0 mm
- net N$3: track 17.8 -> 20.7 mm
- net MY4: track 368.9 -> 371.8 mm
- net N$4: track 16.3 -> 13.6 mm, vias 0 -> 1
- net MX2: track 396.9 -> 398.8 mm
- net MX6: track 463.3 -> 461.5 mm
- net MX0: track 408.5 -> 407.1 mm
- net MX7: track 375.6 -> 374.5 mm
- net N$54: track 18.4 -> 17.8 mm
- net CC2: track 6.91 -> 7.50 mm
Other:
- board size 283.8 x 93.3 mm -> 283.8 x 93.2 mm
- board text added: "1 2 3 4"
- board text added: "Alt | Cmd"
- board text added: "Menu | Opt"
- board text added: "Win | Opt"
- board text removed: "Alt Cmd"
- board text removed: "Menu Opt"
- board text removed: "Win Opt"

Commit message: .
Routing:
- net VBUS: track 25.7 -> 27.9 mm
- net MY0: track 292.6 -> 290.7 mm, vias 9 -> 8
- net MX6: track 461.5 -> 462.3 mm
- net N$4: track 13.6 -> 12.9 mm
