File: EAGLE/vr61/vr61-revB.brd (EAGLE design)
At the start: 283.8 x 93.2 mm, 211 parts, among them M1 M25C, X1 MICROMOD-2222-C

Commit message: .
Parts:
- added U$26: ?, tecsmith_jlcpcb_ordering:JLC_ORDER_NUMBER_QR_5X5
Other:
- board text removed: "JLCJLCJLCJLC"
Changed lines of the file:
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@@
 <setting verticaltext="up"/>
 </settings>
-<grid distance="1.905" unitdist="mm" unit="mm" style="lines" multiple="2" display="yes" altdistance="0.1" altunitdist="mm" altunit="mm"/>
+<grid distance="1" unitdist="mm" unit="mm" style="dots" multiple="2" display="yes" altdistance="0.1" altunitdist="mm" altunit="mm"/>
 <layers>
 <layer number="1" name="Top" color="4" fill="1" visible="yes" active="yes"/>
@@
 <circle x="33.4" y="35.55" radius="2" width="0.5" layer="22"/>
 <circle x="9.45" y="35.55" radius="2" width="0.5" layer="22"/>
-<text x="4.2" y="77.7" size="1.778" layer="22" rot="MR270">JLCJLCJLCJLC</text>
 <circle x="20.6" y="75.8" radius="0.2" width="0.1524" layer="22"/>
 <circle x="41" y="37.6" radius="0.2" width="0.1524" layer="22"/>
@@
 <element name="U$24" library="ts_keyboards" package="FOOTPRINT-BAKENEKO60" value="FOOTPRINT-BAKENEKO60" x="0" y="0" smashed="yes"/>
 <element name="U$25" library="ts_keyboards" package="FOOTPRINT-DIMS-GH60" value="FOOTPRINT-DIMS-GH60" x="0" y="0" smashed="yes"/>
+<element name="U$26" library="tecsmith_jlcpcb_ordering" package="JLC_ORDER_NUMBER_QR_5X5" value="?" x="281" y="4.4" smashed="yes" rot="MR0"/>
 </elements>
 <signals>
