File: EAGLE/vr61/vr61-revC.brd (EAGLE design)
At the start: 283.8 x 93.2 mm, 212 parts, among them M1 M25C, X1 MICROMOD-2222-C

Commit message: Rev C
Parts:
- removed U$25: FOOTPRINT-DIMS-GH60, ts_keyboards:FOOTPRINT-DIMS-GH60
- added S_LALT_2, S_LCTL_2, S_LGUI_2, S_RALT_2, S_RCTL_2, S_RGUI_2, S_SPC_2: MX-5-PIN-HOTSWAP-VIANO-SILK, tecsmith_keyboards:MX-5-PIN-HOTSWAP-VIA-NS
- added U$14: MX-STABS-700U, tecsmith_keyboards:MX-STABS-700U
- added U$27: FOOTPRINT-DIMS-GH60, tecsmith_keyboards:FOOTPRINT-DIMS-GH60
- S_0, S_1, S_2, S_3, S_4, S_5, S_6, S_7, S_8, S_9, S_A, S_APP, S_B, S_BSLS, S_BSPC, S_C, S_CAPS, S_COM, S_D, S_DOT, S_E, S_ENT, S_EQL, S_ESC, S_F, S_FN1, S_G, S_H, S_I, S_J, S_K, S_L, S_LALT, S_LBRC, S_LCTL, S_LGUI, S_LSFT, S_M, S_MINS, S_N, S_O, S_P, S_Q, S_QUOT, S_R, S_RALT, S_RBRC, S_RCTL, S_RSFT, S_S, S_SCLN, S_SLSH, S_SPC, S_T, S_TAB, S_U, S_V, S_W, S_X, S_Y, S_Z: value MX-5-PIN-HOTSWAP-PAD -> MX-5-PIN-HOTSWAP-VIA; device ts_keyboards:MX-5-PIN-HOTSWAP-PAD -> tecsmith_keyboards:MX-5-PIN-HOTSWAP-VIA
- S_BSLS2, S_ENT2, S_LSFT2, S_NUBS: value MX-5-PIN-HOTSWAP-PADNO-SILK -> MX-5-PIN-HOTSWAP-VIANO-SILK; device ts_keyboards:MX-5-PIN-HOTSWAP-PAD-NS -> tecsmith_keyboards:MX-5-PIN-HOTSWAP-VIA-NS
- S_BSPC2, S_FN, S_RSFT2, S_SPARE: value MX-5-PIN-MILMAX-3305-XNO-SILK -> MX-5-PIN-HOTSWAP-VIANO-SILK; device ts_keyboards:MX-5-PIN-MILMAX-3305-X-NS -> tecsmith_keyboards:MX-5-PIN-HOTSWAP-VIA-NS
- S_CAPS2: device ts_keyboards:MX-5-PIN-MILMAX-3305-X-NS -> tecsmith_keyboards:MX-5-PIN-MILMAX-3305-X-NS
- moved U$26 28.3 mm to (281.6, 32.7)
- moved D14 19.0 mm to (245.2, 80.7)
- moved D28 19.0 mm to (245.2, 78.5)
- moved D64 19.0 mm to (245.2, 76.3)
- moved D57 17.9 mm to (46.4, 19.1)
- moved D59 15.8 mm to (211.9, 5.36)
- moved LOGO2 13.1 mm to (190.5, 18.2)
- moved D55 10.6 mm to (23.8, 15.3)
- moved U$8 10.2 mm to (140.2, 16.1)
- moved D56 9.91 mm to (23.8, 13.0)
- moved D60 8.79 mm to (211.9, 7.74)
- moved D54 7.22 mm to (259.4, 20.1)
- moved D61 5.32 mm to (239.4, 7.06)
- moved U$7 4.76 mm to (176.8, 6.00)
- moved D63 4.16 mm to (278.6, 19.3)
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Connections:
- net MY4: now also S_LALT_2.1@1, S_LALT_2.1@2, S_LCTL_2.1@1, S_LCTL_2.1@2, S_LGUI_2.1@1, S_LGUI_2.1@2, S_RALT_2.1@1, S_RALT_2.1@2, S_RCTL_2.1@1, S_RCTL_2.1@2, S_RGUI_2.1@1, S_RGUI_2.1@2, S_SPC_2.1@1, S_SPC_2.1@2
- net MY5: now also S_BSPC2.2@1, S_BSPC2.2@2; no longer S_BSPC2.2
- net MY7: now also S_SPARE.2@1, S_SPARE.2@2; no longer S_SPARE.2
- net MY8: now also S_FN.2@1, S_FN.2@2, S_RSFT2.2@1, S_RSFT2.2@2; no longer S_FN.2, S_RSFT2.2
- net N$14: now also S_BSPC2.1@1, S_BSPC2.1@2; no longer S_BSPC2.1
- net N$53: now also S_RSFT2.1@1, S_RSFT2.1@2; no longer S_RSFT2.1
- net N$54: now also S_LCTL_2.2@1, S_LCTL_2.2@2
- net N$55: now also S_LGUI_2.2@1, S_LGUI_2.2@2
- net N$56: now also S_LALT_2.2@1, S_LALT_2.2@2
- net N$57: now also S_SPC_2.2@1, S_SPC_2.2@2
- net N$59: now also S_RGUI_2.2@1, S_RGUI_2.2@2
- net N$60: now also S_RALT_2.2@1, S_RALT_2.2@2
- net N$61: now also S_RCTL_2.2@1, S_RCTL_2.2@2
- net N$70: now also S_SPARE.1@1, S_SPARE.1@2; no longer S_SPARE.1
- net N$71: now also S_FN.1@1, S_FN.1@2; no longer S_FN.1
Routing:
- net MY4: track 371.8 -> 480.7 mm, vias 4 -> 11
- net MX4: track 468.5 -> 434.5 mm, vias 18 -> 17
- net N$59: track 14.5 -> 44.3 mm, vias 0 -> 2
- net N$60: track 14.2 -> 41.7 mm, vias 0 -> 1
- net N$61: track 14.1 -> 41.5 mm, vias 0 -> 1
- net N$70: track 7.92 -> 31.0 mm
- net N$14: track 32.4 -> 54.9 mm
- net N$57: track 14.8 -> 36.5 mm
- net N$54: track 17.8 -> 39.1 mm
- net MX0: track 407.1 -> 388.6 mm
- net N$28: track 89.6 -> 106.8 mm, vias 3 -> 6
- net MX5: track 381.9 -> 365.0 mm, vias 14 -> 13
- net MX2: track 398.8 -> 382.8 mm
- net MX6: track 462.3 -> 446.3 mm, vias 20 -> 15
- net N$55: track 17.6 -> 30.6 mm, vias 2 -> 1
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Other:
- board text added: "6.25u"
- board text added: "7u"
- board text added: "Rev C | Ver 2024-12-16"
- board text added: "Shft L"
- board text added: "Shft S"
- board text removed: "Rev B.2 | Ver 2024-09-17"
