File: EAGLE/vr61/vr61-revC.sch (EAGLE design)
At the start: 207 parts, among them M1 M25C, X1 MICROMOD-2222-C

Commit message: Rev C
Parts:
- removed U$25: FOOTPRINT-DIMS-GH60, ts_keyboards:FOOTPRINT-DIMS-GH60
- added S_LALT_2, S_LCTL_2, S_LGUI_2, S_RALT_2, S_RCTL_2, S_RGUI_2, S_SPC_2: MX-5-PIN-HOTSWAP-VIANO-SILK, tecsmith_keyboards:MX-5-PIN-HOTSWAP-VIANO-SILK
- added U$14: MX-STABS-700U, tecsmith_keyboards:MX-STABS-700U
- added U$27: FOOTPRINT-DIMS-GH60, tecsmith_keyboards:FOOTPRINT-DIMS-GH60
- S_0, S_1, S_2, S_3, S_4, S_5, S_6, S_7, S_8, S_9, S_A, S_APP, S_B, S_BSLS, S_BSPC, S_C, S_CAPS, S_COM, S_D, S_DOT, S_E, S_ENT, S_EQL, S_ESC, S_F, S_FN1, S_G, S_H, S_I, S_J, S_K, S_L, S_LALT, S_LBRC, S_LCTL, S_LGUI, S_LSFT, S_M, S_MINS, S_N, S_O, S_P, S_Q, S_QUOT, S_R, S_RALT, S_RBRC, S_RCTL, S_RSFT, S_S, S_SCLN, S_SLSH, S_SPC, S_T, S_TAB, S_U, S_V, S_W, S_X, S_Y, S_Z: value MX-5-PIN-HOTSWAP-PAD -> MX-5-PIN-HOTSWAP-VIA; device ts_keyboards:MX-5-PIN-HOTSWAP-PAD -> tecsmith_keyboards:MX-5-PIN-HOTSWAP-VIA
- S_BSLS2, S_ENT2, S_LSFT2, S_NUBS: value MX-5-PIN-HOTSWAP-PADNO-SILK -> MX-5-PIN-HOTSWAP-VIANO-SILK; device ts_keyboards:MX-5-PIN-HOTSWAP-PADNO-SILK -> tecsmith_keyboards:MX-5-PIN-HOTSWAP-VIANO-SILK
- S_BSPC2, S_FN, S_RSFT2, S_SPARE: value MX-5-PIN-MILMAX-3305-XNO-SILK -> MX-5-PIN-HOTSWAP-VIANO-SILK; device ts_keyboards:MX-5-PIN-MILMAX-3305-XNO-SILK -> tecsmith_keyboards:MX-5-PIN-HOTSWAP-VIANO-SILK
- S_CAPS2: device ts_keyboards:MX-5-PIN-MILMAX-3305-XNO-SILK -> tecsmith_keyboards:MX-5-PIN-MILMAX-3305-XNO-SILK
Connections:
- net MY0: now also S_1.1, S_2.1, S_3.1, S_4.1, S_5.1, S_6.1, S_7.1, S_ESC.1; no longer S_1.S, S_2.S, S_3.S, S_4.S, S_5.S, S_6.S, S_7.S, S_ESC.S
- net MY1: now also S_E.1, S_Q.1, S_R.1, S_T.1, S_TAB.1, S_U.1, S_W.1, S_Y.1; no longer S_E.S, S_Q.S, S_R.S, S_T.S, S_TAB.S, S_U.S, S_W.S, S_Y.S
- net MY2: now also S_A.1, S_CAPS.1, S_CAPS2.2, S_D.1, S_F.1, S_G.1, S_H.1, S_J.1, S_S.1; no longer S_A.S, S_CAPS.S, S_CAPS2.P, S_D.S, S_F.S, S_G.S, S_H.S, S_J.S, S_S.S
- net MY3: now also S_B.1, S_C.1, S_LSFT.1, S_LSFT2.1, S_N.1, S_NUBS.1, S_V.1, S_X.1, S_Z.1; no longer S_B.S, S_C.S, S_LSFT.S, S_LSFT2.S, S_N.S, S_NUBS.S, S_V.S, S_X.S, S_Z.S
- net MY4: now also S_APP.1, S_FN1.1, S_LALT.1, S_LALT_2.2, S_LCTL.1, S_LCTL_2.2, S_LGUI.1, S_LGUI_2.2, S_RALT.1, S_RALT_2.2, S_RCTL.1, S_RCTL_2.2, S_RGUI_2.2, S_SPC.1, S_SPC_2.2; no longer S_APP.S, S_FN1.S, S_LALT.S, S_LCTL.S, S_LGUI.S, S_RALT.S, S_RCTL.S, S_SPC.S
- net MY5: now also S_0.1, S_8.1, S_9.1, S_BSPC.1, S_BSPC2.1, S_EQL.1, S_MINS.1; no longer S_0.S, S_8.S, S_9.S, S_BSPC.S, S_BSPC2.S, S_EQL.S, S_MINS.S
- net MY6: now also S_BSLS.1, S_BSLS2.1, S_I.1, S_LBRC.1, S_O.1, S_P.1, S_RBRC.1; no longer S_BSLS.S, S_BSLS2.S, S_I.S, S_LBRC.S, S_O.S, S_P.S, S_RBRC.S
- net MY7: now also S_ENT.1, S_ENT2.1, S_K.1, S_L.1, S_QUOT.1, S_SCLN.1, S_SPARE.1; no longer S_ENT.S, S_ENT2.S, S_K.S, S_L.S, S_QUOT.S, S_SCLN.S, S_SPARE.S
- net MY8: now also S_COM.1, S_DOT.1, S_FN.1, S_M.1, S_RSFT.1, S_RSFT2.1, S_SLSH.1; no longer S_COM.S, S_DOT.S, S_FN.S, S_M.S, S_RSFT.S, S_RSFT2.S, S_SLSH.S
- net N$1: now also S_ESC.2; no longer S_ESC.P
- net N$10: now also S_9.2; no longer S_9.P
- net N$11: now also S_0.2; no longer S_0.P
- net N$12: now also S_MINS.2; no longer S_MINS.P
- net N$13: now also S_EQL.2; no longer S_EQL.P
- net N$14: now also S_BSPC.2, S_BSPC2.2; no longer S_BSPC.P, S_BSPC2.P
- net N$15: now also S_TAB.2; no longer S_TAB.P
- net N$16: now also S_Q.2; no longer S_Q.P
- net N$17: now also S_W.2; no longer S_W.P
- net N$18: now also S_E.2; no longer S_E.P
- net N$19: now also S_R.2; no longer S_R.P
- net N$2: now also S_1.2; no longer S_1.P
- net N$20: now also S_T.2; no longer S_T.P
- net N$21: now also S_Y.2; no longer S_Y.P
- net N$22: now also S_U.2; no longer S_U.P
- net N$23: now also S_I.2; no longer S_I.P
- net N$24: now also S_O.2; no longer S_O.P
- net N$25: now also S_P.2; no longer S_P.P
- net N$26: now also S_LBRC.2; no longer S_LBRC.P
- net N$27: now also S_RBRC.2; no longer S_RBRC.P
- net N$28: now also S_BSLS.2, S_BSLS2.2; no longer S_BSLS.P, S_BSLS2.P
- net N$3: now also S_2.2; no longer S_2.P
- net N$30: now also S_A.2; no longer S_A.P
- net N$31: now also S_S.2; no longer S_S.P
- net N$32: now also S_D.2; no longer S_D.P
- net N$33: now also S_F.2; no longer S_F.P
- net N$34: now also S_G.2; no longer S_G.P
- net N$35: now also S_H.2; no longer S_H.P
- net N$36: now also S_J.2; no longer S_J.P
- net N$37: now also S_K.2; no longer S_K.P
- net N$38: now also S_L.2; no longer S_L.P
- net N$39: now also S_SCLN.2; no longer S_SCLN.P
- net N$4: now also S_3.2; no longer S_3.P
- net N$40: now also S_QUOT.2; no longer S_QUOT.P
- net N$41: now also S_ENT.2, S_ENT2.2; no longer S_ENT.P, S_ENT2.P
- net N$42: now also S_LSFT.2, S_LSFT2.2; no longer S_LSFT.P, S_LSFT2.P
- net N$43: now also S_Z.2; no longer S_Z.P
- net N$44: now also S_X.2; no longer S_X.P
- net N$45: now also S_C.2; no longer S_C.P
- net N$46: now also S_V.2; no longer S_V.P
- net N$47: now also S_B.2; no longer S_B.P
- net N$48: now also S_N.2; no longer S_N.P
- net N$49: now also S_M.2; no longer S_M.P
- net N$5: now also S_4.2; no longer S_4.P
- net N$50: now also S_COM.2; no longer S_COM.P
- net N$51: now also S_DOT.2; no longer S_DOT.P
- net N$52: now also S_SLSH.2; no longer S_SLSH.P
- net N$53: now also S_RSFT.2, S_RSFT2.2; no longer S_RSFT.P, S_RSFT2.P
- net N$54: now also S_LCTL.2, S_LCTL_2.1; no longer S_LCTL.P
- net N$55: now also S_LGUI.2, S_LGUI_2.1; no longer S_LGUI.P
- net N$56: now also S_LALT.2, S_LALT_2.1; no longer S_LALT.P
- net N$57: now also S_SPC.2, S_SPC_2.1; no longer S_SPC.P
- net N$58: now also S_FN1.2; no longer S_FN1.P
- net N$59: now also S_APP.2, S_RGUI_2.1; no longer S_APP.P
- net N$6: now also S_5.2; no longer S_5.P
- net N$60: now also S_RALT.2, S_RALT_2.1; no longer S_RALT.P
- net N$61: now also S_RCTL.2, S_RCTL_2.1; no longer S_RCTL.P
- net N$62: now also S_CAPS.2, S_CAPS2.1; no longer S_CAPS.P, S_CAPS2.S
- net N$69: now also S_NUBS.2; no longer S_NUBS.P
- net N$7: now also S_6.2; no longer S_6.P
- net N$70: now also S_SPARE.2; no longer S_SPARE.P
- net N$71: now also S_FN.2; no longer S_FN.P
- net N$8: now also S_7.2; no longer S_7.P
- net N$9: now also S_8.2; no longer S_8.P
Other:
- moved on the sheet: S_0, S_1, S_2, S_3, S_4, S_5, S_6, S_7, S_8, S_9, S_A, S_APP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
