File: EAGLE/c3-udb/c3-udb.brd (EAGLE design)
At the start: 18 x 16.5 mm, 11 parts, among them J2 SM04B-SRSS-TB(LF)(SN), X1 TYPE-C-31-M-12, Y1 ESD_TPD4E05U06

Commit message: update udb
Parts:
- added J1: (no value), __untitled:1X04_SMD_RA_FEMALE
- LOGO1: value OSHW-LOGOM -> OSHW-LOGOS; device random_logos:OSHW-LOGO-M -> SparkFun-Aesthetics:OSHW-LOGO-S
- moved LOGO1 10.1 mm to (16.0, 5.70)
Connections:
- net D+: now also J1.3
- net D-: now also J1.2
- net GND: now also J1.4
- net VSUP: now also J1.1
Routing:
- net D+: track 11.9 -> 15.8 mm
- net VSUP: track 16.3 -> 19.5 mm, vias 0 -> 1
- net GND: track 9.86 -> 12.9 mm, vias 4 -> 3
- net D-: track 12.9 -> 15.4 mm
Other:
- board text added: "5V"
- board text added: "D+"
- board text added: "D-"
- board text added: "GND"
- board text added: "Original (c) 2019 @ai03"
- board text removed: "Original (c) ai03"
Changed lines of the file:
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@@
 <wire x1="18" y1="2" x2="16" y2="0" width="0.0762" layer="20" curve="-88.492564"/>
 <text x="14.1" y="5.8" size="0.6096" layer="21" rot="R270">PTC</text>
-<text x="2.5" y="8.2" size="0.8128" layer="22" rot="MR90" align="center">Unified
+<text x="2" y="8.2" size="0.8128" layer="22" rot="MR90" align="center">Unified
 Daughterboard</text>
-<text x="16.1" y="8" size="0.6096" layer="22" rot="MR90" align="center">http://c1k.it/udb</text>
-<text x="12.5" y="3.5" size="0.6096" layer="22" rot="MR90" align="center">Original
-(c) ai03</text>
+<text x="9" y="16" size="0.6096" layer="22" rot="MR0" align="center">http://c1k.it/udb</text>
+<text x="16" y="10" size="0.6096" layer="22" rot="MR90" align="center">Original
+(c) 2019
+@ai03</text>
 <text x="6.4" y="14.9" size="0.6096" layer="22" rot="MR90" align="center-right">a clone by
 Tecsmith</text>
+<text x="5.2" y="3.85" size="0.6096" layer="26" ratio="20" rot="MR90" align="center-left">GND</text>
+<text x="7.7" y="3.85" size="0.6096" layer="26" ratio="20" rot="MR90" align="center-left">D-</text>
+<text x="10.2" y="3.85" size="0.6096" layer="26" ratio="20" rot="MR90" align="center-left">D+</text>
+<text x="12.7" y="3.85" size="0.6096" layer="26" ratio="20" rot="MR90" align="center-left">5V</text>
 </plain>
 <attributes>
@@
 </class>
 </classes>
-<designrules name="default">
+<designrules name="default *">
 <description language="de">&lt;b&gt;EAGLE Design Rules&lt;/b&gt;
 &lt;p&gt;
@@
 <param name="mdSmdStop" value="0mil"/>
 <param name="msWidth" value="6mil"/>
-<param name="msDrill" value="0.35mm"/>
+<param name="msDrill" value="0.3mm"/>
 <param name="msMicroVia" value="9.99mm"/>
 <param name="msBlindViaRatio" value="0.5"/>
@@
 </element>
 <element name="U$2" library="random_logos" package="TECSMITH-CUBE" value="TECSMITH-LOGOSHORT" x="10" y="12.7" smashed="yes" rot="MR90"/>
-<element name="LOGO1" library="random_logos" package="OSHW-LOGO-M" value="OSHW-LOGOM" x="6.1" y="3.5" smashed="yes" rot="MR90"/>
+<element name="LOGO1" library="SparkFun-Aesthetics" library_urn="urn:adsk.eagle:library:507" package="OSHW-LOGO-S" package3d_urn="urn:adsk.eagle:package:37099/1" value="OSHW-LOGOS" x="16" y="5.7" smashed="yes" rot="MR90"/>
+<element name="J1" library="__untitled" package="1X04_SMD_RA_FEMALE" package3d_urn="urn:adsk.eagle:package:38100/1" value="" x="9" y="2" smashed="yes" rot="MR0">
+<attribute name="PROD_ID" value="CONN-12382" x="9" y="2" size="1.778" layer="28" rot="MR0" display="off"/>
+</element>
 </elements>
 <signals>
@@
 <contactref element="R1" pad="2"/>
 <contactref element="R2" pad="2"/>
-<via x="9" y="8.1" extent="1-16" drill="0.35" diameter="0.55"/>
+<via x="9" y="8.1" extent="1-16" drill="0.3" diameter="0.55"/>
 <wire x1="9" y1="8.1" x2="9" y2="5.8" width="0.254" layer="1"/>
 <polygon width="0.0762" layer="1">
@@
 <vertex x="0" y="0"/>
 </polygon>
-<via x="4" y="7" extent="1-16" drill="0.35"/>
-<via x="9" y="2" extent="1-16" drill="0.35"/>
-<via x="13.4" y="6" extent="1-16" drill="0.35"/>
+<via x="4" y="7" extent="1-16" drill="0.3"/>
+<via x="14" y="6.5" extent="1-16" drill="0.3"/>
 <polygon width="0.0762" layer="16">
 <vertex x="0" y="0"/>
+<vertex x="6" y="0"/>
+<vertex x="6" y="4"/>
+<vertex x="12" y="4"/>
+<vertex x="12" y="0"/>
 <vertex x="18" y="0"/>
 <vertex x="18" y="8.5"/>
@@
 <wire x1="16.02" y1="9.88" x2="15.94" y2="9.8" width="0.508" layer="1"/>
 <wire x1="15.94" y1="9.8" x2="14.6" y2="9.8" width="0.508" layer="1"/>
+<contactref element="J1" pad="4"/>
+<wire x1="5.19" y1="2" x2="5.19" y2="5.04" width="0.508" layer="16"/>
 </signal>
 <signal name="VSUP">
@@
 <wire x1="4.1" y1="5" x2="5.7" y2="3.4" width="0.508" layer="1"/>
 <wire x1="5.7" y1="3.4" x2="7.5" y2="3.4" width="0.508" layer="1"/>
-<wire x1="7.5" y1="3.4" x2="12.3" y2="3.4" width="0.508" layer="1"/>
-<wire x1="13.79" y1="4.89" x2="15.81" y2="4.89" width="0.508" layer="1"/>
-<wire x1="12.3" y1="3.4" x2="13.79" y2="4.89" width="0.508" layer="1"/>
 <wire x1="7.5" y1="4.7" x2="7.5" y2="3.4" width="0.508" layer="1"/>
+<via x="13.7" y="4.45" extent="1-16" drill="0.35"/>
+<wire x1="12.65" y1="3.4" x2="13.7" y2="4.45" width="0.508" layer="1"/>
+<wire x1="7.5" y1="3.4" x2="12.65" y2="3.4" width="0.508" layer="1"/>
+<wire x1="13.7" y1="4.45" x2="14.14" y2="4.89" width="0.508" layer="1"/>
+<wire x1="14.14" y1="4.89" x2="15.81" y2="4.89" width="0.508" layer="1"/>
+<contactref element="J1" pad="1"/>
+<wire x1="12.81" y1="2" x2="12.81" y2="4.06" width="0.508" layer="16"/>
+<wire x1="13.2" y1="4.45" x2="12.81" y2="4.06" width="0.508" layer="16"/>
+<wire x1="13.2" y1="4.45" x2="13.7" y2="4.45" width="0.508" layer="16"/>
 </signal>
 <signal name="CC1">
@@
 <wire x1="9.66" y1="7.84" x2="9.5" y2="7.68" width="0.254" layer="1"/>
 <wire x1="9.5" y1="7.68" x2="9.5" y2="4.7" width="0.254" layer="1"/>
-<via x="9.5" y="4.7" extent="1-16" drill="0.35"/>
+<via x="9.5" y="4.7" extent="1-16" drill="0.3"/>
 <wire x1="8.25" y1="9.59" x2="8.25" y2="8.86" width="0.254" layer="1"/>
 <wire x1="8" y1="7.6175" x2="7.93" y2="7.6875" width="0.254" layer="1"/>
@@
 <wire x1="7.93" y1="8.54" x2="7.93" y2="7.6875" width="0.254" layer="1"/>
 <wire x1="8" y1="6.4" x2="7.6" y2="6" width="0.254" layer="1"/>
-<via x="7.6" y="6" extent="1-16" drill="0.35"/>
+<via x="7.6" y="6" extent="1-16" drill="0.3"/>
 <wire x1="8" y1="7.4175" x2="8" y2="6.4" width="0.254" layer="1"/>
-<wire x1="7.6" y1="6" x2="8.84" y2="6" width="0.254" layer="16"/>
-<wire x1="9.5" y1="5.34" x2="8.84" y2="6" width="0.254" layer="16"/>
-<wire x1="9.5" y1="5.34" x2="9.5" y2="4.7" width="0.254" layer="16"/>
+<wire x1="7.6" y1="6" x2="8.1" y2="5.5" width="0.254" layer="16"/>
+<wire x1="9.14" y1="5.5" x2="8.1" y2="5.5" width="0.254" layer="16"/>
+<wire x1="9.5" y1="5.14" x2="9.14" y2="5.5" width="0.254" layer="16"/>
+<wire x1="9.5" y1="5.14" x2="9.5" y2="4.7" width="0.254" layer="16"/>
+<contactref element="J1" pad="3"/>
+<wire x1="7.6" y1="6" x2="7.6" y2="3.78" width="0.254" layer="16"/>
+<wire x1="7.73" y1="3.65" x2="7.6" y2="3.78" width="0.254" layer="16"/>
+<wire x1="7.73" y1="3.65" x2="7.73" y2="2" width="0.254" layer="16"/>
 <wire x1="8" y1="7.4175" x2="9.5" y2="7.4175" width="0" layer="19" extent="1-1"/>
 </signal>
@@
 <wire x1="8.34" y1="7.8375" x2="8.34" y2="8.37" width="0.254" layer="1"/>
 <wire x1="8.5" y1="7.4175" x2="8.5" y2="4.7" width="0.254" layer="1"/>
-<via x="8.5" y="4.7" extent="1-16" drill="0.35"/>
+<via x="8.5" y="4.7" extent="1-16" drill="0.3" diameter="0.5"/>
 <wire x1="9.75" y1="9.59" x2="9.75" y2="8.86" width="0.254" layer="1"/>
 <wire x1="10.07" y1="7.6875" x2="10" y2="7.6175" width="0.254" layer="1"/>
@@
 <wire x1="10.07" y1="8.54" x2="10.07" y2="7.6875" width="0.254" layer="1"/>
 <wire x1="10" y1="6.4" x2="10.4" y2="6" width="0.254" layer="1"/>
-<via x="10.4" y="6" extent="1-16" drill="0.35"/>
+<via x="10.4" y="6" extent="1-16" drill="0.3"/>
 <wire x1="10" y1="7.4175" x2="10" y2="6.4" width="0.254" layer="1"/>
-<wire x1="8.5" y1="4.7" x2="9.2" y2="4" width="0.254" layer="16"/>
-<wire x1="10.4" y1="4.6" x2="10.4" y2="6" width="0.254" layer="16"/>
-<wire x1="9.2" y1="4" x2="9.8" y2="4" width="0.254" layer="16"/>
-<wire x1="9.8" y1="4" x2="10.4" y2="4.6" width="0.254" layer="16"/>
+<wire x1="9.1" y1="3.9" x2="8.5" y2="4.5" width="0.254" layer="16"/>
+<wire x1="8.5" y1="4.7" x2="8.5" y2="4.5" width="0.254" layer="16"/>
+<wire x1="10.4" y1="4.45" x2="10.4" y2="6" width="0.254" layer="16"/>
+<wire x1="9.1" y1="3.9" x2="9.85" y2="3.9" width="0.254" layer="16"/>
+<wire x1="9.85" y1="3.9" x2="10.1" y2="4.15" width="0.254" layer="16"/>
+<contactref element="J1" pad="2"/>
+<wire x1="10.1" y1="4.15" x2="10.4" y2="4.45" width="0.254" layer="16"/>
+<wire x1="10.27" y1="2" x2="10.27" y2="3.98" width="0.254" layer="16"/>
+<wire x1="10.27" y1="3.98" x2="10.1" y2="4.15" width="0.254" layer="16"/>
 </signal>
 <signal name="VBUS">
@@
 <vertex x="18" y="16.5"/>
 </polygon>
-<wire x1="13.32" y1="10.16" x2="16.02" y2="11.58" width="0" layer="19" extent="1-1"/>
-<wire x1="4.68" y1="10.16" x2="13.32" y2="10.16" width="0" layer="19" extent="1-1"/>
-<wire x1="1.96" y1="11.58" x2="4.68" y2="10.16" width="0" layer="19" extent="1-1"/>
 </signal>
 </signals>
