File: EAGLE/c3-udb/c3-udb.sch (EAGLE design)
At the start: 11 parts, among them J2 SM04B-SRSS-TB(LF)(SN), X1 TYPE-C-31-M-12, Y1 ESD_TPD4E05U06

Commit message: update udb
Parts:
- added J1: (no value), __untitled:CONN_04SMD_RA_FEMALE
- LOGO1: value OSHW-LOGOM -> OSHW-LOGOS; device random_logos:OSHW-LOGOM -> SparkFun-Aesthetics:OSHW-LOGOS
Connections:
- net D+: now also J1.3
- net D-: now also J1.2
- net GND: now also J1.4
- net VSUP: now also J1.1
Other:
- moved on the sheet: J2
Changed lines of the file:
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@@
 <part name="R2" library="rcl" library_urn="urn:adsk.eagle:library:334" deviceset="R-EU_" device="R0402" package3d_urn="urn:adsk.eagle:package:23547/3" value="5.1K"/>
 <part name="U$2" library="random_logos" deviceset="TECSMITH-LOGO" device="SHORT"/>
-<part name="LOGO1" library="random_logos" deviceset="OSHW-LOGO" device="M"/>
+<part name="LOGO1" library="SparkFun-Aesthetics" library_urn="urn:adsk.eagle:library:507" deviceset="OSHW-LOGO" device="S" package3d_urn="urn:adsk.eagle:package:37099/1"/>
+<part name="J1" library="__untitled" deviceset="CONN_04" device="SMD_RA_FEMALE" package3d_urn="urn:adsk.eagle:package:38100/1"/>
 </parts>
 <sheets>
@@
 <attribute name="VALUE" x="73.66" y="88.9" size="1.27" layer="96"/>
 </instance>
-<instance part="U$11" gate="G$1" x="144.78" y="116.84" smashed="yes">
-<attribute name="VALUE" x="144.78" y="121.412" size="1.778" layer="96" align="bottom-center"/>
+<instance part="U$11" gate="G$1" x="144.78" y="127" smashed="yes">
+<attribute name="VALUE" x="144.78" y="131.572" size="1.778" layer="96" align="bottom-center"/>
 </instance>
 <instance part="GND4" gate="1" x="101.6" y="66.04" smashed="yes">
 <attribute name="VALUE" x="101.6" y="61.468" size="1.778" layer="96" align="top-center"/>
 </instance>
-<instance part="J2" gate="J1" x="160.02" y="111.76" smashed="yes" rot="R180">
-<attribute name="VALUE" x="164.846" y="99.06" size="1.778" layer="96" font="vector" rot="R270" align="top-left"/>
-<attribute name="NAME" x="165.1" y="103.886" size="1.778" layer="95" font="vector" rot="R180"/>
+<instance part="J2" gate="J1" x="170.18" y="111.76" smashed="yes" rot="R180">
+<attribute name="VALUE" x="175.006" y="99.06" size="1.778" layer="96" font="vector" rot="R270" align="top-left"/>
+<attribute name="NAME" x="175.26" y="103.886" size="1.778" layer="95" font="vector" rot="R180"/>
 </instance>
 <instance part="R3" gate="G$1" x="83.82" y="78.74" smashed="yes" rot="R90">
@@
 <attribute name="VALUE" x="105.41" y="93.218" size="1.778" layer="96"/>
 </instance>
-<instance part="U$2" gate="G$1" x="254" y="27.94" smashed="yes"/>
-<instance part="LOGO1" gate="G$1" x="254" y="25.4" smashed="yes"/>
+<instance part="U$2" gate="G$1" x="7.62" y="20.32" smashed="yes"/>
+<instance part="LOGO1" gate="G$1" x="12.7" y="10.16" smashed="yes"/>
+<instance part="J1" gate="G$1" x="154.94" y="121.92" smashed="yes" rot="R270">
+<attribute name="VALUE" x="147.574" y="127" size="1.778" layer="96" font="vector" rot="R270"/>
+<attribute name="NAME" x="163.068" y="127" size="1.778" layer="95" font="vector" rot="R270"/>
+</instance>
 </instances>
 <busses>
@@
 <wire x1="116.84" y1="83.82" x2="101.6" y2="83.82" width="0.1524" layer="91"/>
 <junction x="101.6" y="83.82"/>
-<wire x1="152.4" y1="106.68" x2="149.86" y2="106.68" width="0.1524" layer="91"/>
+<wire x1="162.56" y1="106.68" x2="160.02" y2="106.68" width="0.1524" layer="91"/>
 <pinref part="J2" gate="J1" pin="GND"/>
+<wire x1="160.02" y1="106.68" x2="149.86" y2="106.68" width="0.1524" layer="91"/>
 <wire x1="149.86" y1="106.68" x2="149.86" y2="83.82" width="0.1524" layer="91"/>
 <wire x1="149.86" y1="83.82" x2="144.78" y2="83.82" width="0.1524" layer="91"/>
@@
 <pinref part="R1" gate="G$1" pin="2"/>
 <pinref part="R2" gate="G$1" pin="2"/>
+<wire x1="160.02" y1="116.84" x2="160.02" y2="106.68" width="0.1524" layer="91"/>
+<junction x="160.02" y="106.68"/>
+<pinref part="J1" gate="G$1" pin="4"/>
 </segment>
 </net>
@@
 <segment>
 <pinref part="U$11" gate="G$1" pin="VCC"/>
-<wire x1="144.78" y1="116.84" x2="144.78" y2="114.3" width="0.1524" layer="91"/>
+<wire x1="144.78" y1="127" x2="144.78" y2="114.3" width="0.1524" layer="91"/>
 <pinref part="PTC" gate="G$1" pin="2"/>
 <wire x1="114.3" y1="114.3" x2="144.78" y2="114.3" width="0.1524" layer="91"/>
@@
 <junction x="144.78" y="114.3"/>
 <pinref part="J2" gate="J1" pin="VCC"/>
+<wire x1="162.56" y1="114.3" x2="152.4" y2="114.3" width="0.1524" layer="91"/>
 <wire x1="152.4" y1="114.3" x2="144.78" y2="114.3" width="0.1524" layer="91"/>
+<wire x1="152.4" y1="116.84" x2="152.4" y2="114.3" width="0.1524" layer="91"/>
+<junction x="152.4" y="114.3"/>
+<pinref part="J1" gate="G$1" pin="1"/>
 </segment>
 </net>
@@
 <wire x1="147.32" y1="111.76" x2="149.86" y2="109.22" width="0.1524" layer="91"/>
 <pinref part="J2" gate="J1" pin="D+"/>
-<wire x1="149.86" y1="109.22" x2="152.4" y2="109.22" width="0.1524" layer="91"/>
+<wire x1="149.86" y1="109.22" x2="157.48" y2="109.22" width="0.1524" layer="91"/>
 <pinref part="Y1" gate="G$1" pin="D2-"/>
+<wire x1="157.48" y1="109.22" x2="162.56" y2="109.22" width="0.1524" layer="91"/>
 <wire x1="124.46" y1="101.6" x2="124.46" y2="111.76" width="0.1524" layer="91"/>
 <junction x="124.46" y="111.76"/>
@@
 <wire x1="132.08" y1="101.6" x2="132.08" y2="111.76" width="0.1524" layer="91"/>
 <junction x="132.08" y="111.76"/>
+<wire x1="157.48" y1="116.84" x2="157.48" y2="109.22" width="0.1524" layer="91"/>
+<junction x="157.48" y="109.22"/>
+<pinref part="J1" gate="G$1" pin="3"/>
 </segment>
 </net>
@@
 <segment>
 <pinref part="J2" gate="J1" pin="D-"/>
-<wire x1="152.4" y1="111.76" x2="149.86" y2="111.76" width="0.1524" layer="91"/>
+<wire x1="162.56" y1="111.76" x2="154.94" y2="111.76" width="0.1524" layer="91"/>
+<wire x1="154.94" y1="111.76" x2="149.86" y2="111.76" width="0.1524" layer="91"/>
 <wire x1="149.86" y1="111.76" x2="147.32" y2="109.22" width="0.1524" layer="91"/>
 <pinref part="X1" gate="G$1" pin="D-"/>
@@
 <wire x1="134.62" y1="101.6" x2="134.62" y2="109.22" width="0.1524" layer="91"/>
 <junction x="134.62" y="109.22"/>
+<wire x1="154.94" y1="116.84" x2="154.94" y2="111.76" width="0.1524" layer="91"/>
+<junction x="154.94" y="111.76"/>
+<pinref part="J1" gate="G$1" pin="2"/>
 </segment>
 </net>
